File: BMS/Battery_0-12.kicad_sch (KiCad schematic)
At the start: 69 parts, among them J1 Conn_01x17, J12 Conn_01x17

Commit message: zmiany w bq79614 layout
Connections:
- net Batt_Coupling: now also J1.17 (Pin_17); no longer J1.14 (Pin_14)
- net GND_HV: now also J1.4 (Pin_4); no longer J1.1 (Pin_1)
- net at BT7.2 (-), BT8.1 (+), R27.1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: now also J1.10 (Pin_10); no longer J1.7 (Pin_7)
- net at BT8.2 (-), BT9.1 (+), R28.1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: now also J1.9 (Pin_9); no longer J1.6 (Pin_6)
- net at BT6.2 (-), BT7.1 (+), R26.1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: now also J1.11 (Pin_11); no longer J1.8 (Pin_8)
- net at BT1.2 (-), BT2.1 (+), R21.1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: now also J1.16 (Pin_16); no longer J1.13 (Pin_13)
- net at BT12.2 (-), BT13.1 (+), R32.1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: now also J1.5 (Pin_5); no longer J1.2 (Pin_2)
- net at BT11.2 (-), BT12.1 (+), R31.1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: now also J1.6 (Pin_6); no longer J1.3 (Pin_3)
- net at BT10.2 (-), BT11.1 (+), R30.1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: now also J1.7 (Pin_7); no longer J1.4 (Pin_4)
- net at BT10.1 (+), BT9.2 (-), R29.1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: now also J1.8 (Pin_8); no longer J1.5 (Pin_5)
- net at BT4.2 (-), BT5.1 (+), R24.1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: now also J1.13 (Pin_13); no longer J1.10 (Pin_10)
- net at BT5.2 (-), BT6.1 (+), R25.1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: now also J1.12 (Pin_12); no longer J1.9 (Pin_9)
- net at BT3.2 (-), BT4.1 (+), R23.1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: now also J1.14 (Pin_14); no longer J1.11 (Pin_11)
- net at BT2.2 (-), BT3.1 (+), R22.1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: now also J1.15 (Pin_15); no longer J1.12 (Pin_12)
Changed lines of the file:
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@@
 	)
 	(no_connect
-		(at 26.67 99.06)
+		(at 26.67 144.78)
 	)
 	(no_connect
@@
 	)
 	(no_connect
-		(at 26.67 101.6)
-	)
-	(no_connect
 		(at 26.67 46.99)
 	)
@@
 	)
 	(no_connect
-		(at 26.67 96.52)
+		(at 26.67 142.24)
+	)
+	(no_connect
+		(at 26.67 139.7)
 	)
 	(wire
@@
 	)
 	(symbol
-		(lib_id "Connector_Generic:Conn_01x17")
-		(at 21.59 116.84 180)
-		(unit 1)
-		(exclude_from_sim no)
-		(in_bom yes)
-		(on_board yes)
-		(dnp no)
-		(fields_autoplaced yes)
-		(property "Reference" "J1"
-			(at 21.59 90.17 0)
-			(effects
-				(font
-					(size 1.27 1.27)
-				)
-			)
-		)
-		(property "Value" "Conn_01x17"
-			(at 21.59 92.71 0)
-			(effects
-				(font
-					(size 1.27 1.27)
-				)
-			)
-		)
-		(property "Footprint" "footrpint:HARWIN_B5743-117-M-L-1"
-			(at 21.59 116.84 0)
-			(effects
-				(font
-					(size 1.27 1.27)
-				)
-				(hide yes)
-			)
-		)
-		(property "Datasheet" "https://www.harwin.com/products/B5743-117-M-L-1"
-			(at 21.59 116.84 0)
-			(effects
-				(font
-					(size 1.27 1.27)
-				)
-				(hide yes)
-			)
-		)
-		(property "Description" "Generic connector, single row, 01x17, script generated (kicad-library-utils/schlib/autogen/connector/)"
-			(at 21.59 116.84 0)
-			(effects
-				(font
-					(size 1.27 1.27)
-				)
-				(hide yes)
-			)
-		)
-		(pin "13"
-		)
-		(pin "17"
-		)
-		(pin "3"
-		)
-		(pin "4"
-		)
-		(pin "10"
-		)
-		(pin "14"
-		)
-		(pin "16"
-		)
-		(pin "11"
-		)
-		(pin "1"
-		)
-		(pin "12"
-		)
-		(pin "5"
-		)
-		(pin "9"
-		)
-		(pin "8"
-		)
-		(pin "15"
-		)
-		(pin "6"
-		)
-		(pin "2"
-		)
-		(pin "7"
-		)
-		(instances
-			(project "BMS"
-				(path "/26289bb6-56bc-4ca1-b1a2-18d58d1afdf5/329d2a9a-b359-4d8c-80ce-edb0b764c6b7/1b0b9d23-485d-43ce-ac65-957d0a9baa65"
-					(reference "J1")
-					(unit 1)
-				)
-			)
-		)
-	)
-	(symbol
 		(lib_id "Device:Battery_Cell")
 		(at 95.25 144.78 0)
@@
 					(unit 1)
 				)
+				(path "/26289bb6-56bc-4ca1-b1a2-18d58d1afdf5/329d2a9a-b359-4d8c-80ce-edb0b764c6b7/a43b6b0a-d3da-47c5-ab92-e0e154337573"
+					(reference "R38")
+					(unit 1)
+				)
 			)
 		)
@@
 					(unit 1)
 				)
+			)
+		)
+	)
+	(symbol
+		(lib_id "Connector_Generic:Conn_01x17")
+		(at 21.59 124.46 180)
+		(unit 1)
+		(exclude_from_sim no)
+		(in_bom yes)
+		(on_board yes)
+		(dnp no)
+		(fields_autoplaced yes)
+		(property "Reference" "J1"
+			(at 21.59 97.79 0)
+			(effects
+				(font
+					(size 1.27 1.27)
+				)
+			)
+		)
+		(property "Value" "Conn_01x17"
+			(at 21.59 100.33 0)
+			(effects
+				(font
+					(size 1.27 1.27)
+				)
+			)
+		)
+		(property "Footprint" "footrpint:HARWIN_B5743-117-M-L-1"
+			(at 21.59 124.46 0)
+			(effects
+				(font
+					(size 1.27 1.27)
+				)
+				(hide yes)
+			)
+		)
+		(property "Datasheet" "https://www.harwin.com/products/B5743-117-M-L-1"
+			(at 21.59 124.46 0)
+			(effects
+				(font
+					(size 1.27 1.27)
+				)
+				(hide yes)
+			)
+		)
+		(property "Description" "Generic connector, single row, 01x17, script generated (kicad-library-utils/schlib/autogen/connector/)"
+			(at 21.59 124.46 0)
+			(effects
+				(font
+					(size 1.27 1.27)
+				)
+				(hide yes)
+			)
+		)
+		(pin "13"
+		)
+		(pin "17"
+		)
+		(pin "3"
+		)
+		(pin "4"
+		)
+		(pin "10"
+		)
+		(pin "14"
+		)
+		(pin "16"
+		)
+		(pin "11"
+		)
+		(pin "1"
+		)
+		(pin "12"
+		)
+		(pin "5"
+		)
+		(pin "9"
+		)
+		(pin "8"
+		)
+		(pin "15"
+		)
+		(pin "6"
+		)
+		(pin "2"
+		)
+		(pin "7"
+		)
+		(instances
+			(project "BMS"
+				(path "/26289bb6-56bc-4ca1-b1a2-18d58d1afdf5/329d2a9a-b359-4d8c-80ce-edb0b764c6b7/1b0b9d23-485d-43ce-ac65-957d0a9baa65"
+					(reference "J1")
+					(unit 1)
+				)
