File: BMS/Mesurements_LTC1.kicad_sch (KiCad schematic)
At the start: 12 parts, among them Q1 NPN, U1 BQ79614PAPRQ1

Commit message: zmiany w bq79614 layout
Connections:
- net GND_HV: now also C9.1, U1.39 (AVSS)
