File: BMS/Mesurements_LTC2.kicad_sch (KiCad schematic)
At the start: 12 parts, among them Q2 NPN, U2 BQ79614PAPRQ1

Commit message: Iteracja 1.0 gotowa, teraz sprawdzenie i zmiany kosmetyczne
Parts:
- R64: value 300 -> 300
Changed lines of the file:
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@@
 (kicad_sch
-	(version 20231120)
+	(version 20250114)
 	(generator "eeschema")
-	(generator_version "8.0")
+	(generator_version "9.0")
 	(paper "A4")
+	(text "sprwadzic to\n"
+		(exclude_from_sim no)
+		(at 150.876 131.064 0)
+		(effects
+			(font
+				(size 1.27 1.27)
+			)
+		)
+	)
+	(text "max 370ohm\n"
+		(exclude_from_sim no)
+		(at 51.562 78.486 0)
+		(effects
+			(font
+				(size 1.27 1.27)
+			)
+		)
+	)
+	(text "NPNB DO SPRAWDZENIA (DOBRAC REZYSTORY)\n"
+		(exclude_from_sim no)
+		(at 36.322 61.722 0)
+		(effects
+			(font
+				(size 1.27 1.27)
+			)
+		)
+	)
 	(junction
 		(at 78.74 78.74)
@@
 		)
 	)
-	(text "sprwadzic to\n"
-		(exclude_from_sim no)
-		(at 150.876 131.064 0)
-		(effects
-			(font
-				(size 1.27 1.27)
-			)
-		)
-	)
-	(text "max 370ohm\n"
-		(exclude_from_sim no)
-		(at 51.562 78.486 0)
-		(effects
-			(font
-				(size 1.27 1.27)
-			)
-		)
-	)
-	(text "NPNB DO SPRAWDZENIA (DOBRAC REZYSTORY)\n"
-		(exclude_from_sim no)
-		(at 36.322 61.722 0)
-		(effects
-			(font
-				(size 1.27 1.27)
-			)
-		)
-	)
 	(label "VC0"
 		(at 27.94 132.08 0)
-		(fields_autoplaced yes)
 		(effects
 			(font
@@
 	(label "CB11"
 		(at 64.77 104.14 180)
-		(fields_autoplaced yes)
 		(effects
 			(font
@@
 	(label "CB11"
 		(at 143.51 46.99 180)
-		(fields_autoplaced yes)
 		(effects
 			(font
@@
 	(label "VC10"
 		(at 85.09 102.87 0)
-		(fields_autoplaced yes)
 		(effects
 			(font
@@
 	(label "CB1"
 		(at 143.51 72.39 180)
-		(fields_autoplaced yes)
 		(effects
 			(font
@@
 	(label "CB6"
 		(at 64.77 116.84 180)
-		(fields_autoplaced yes)
 		(effects
 			(font
@@
 	(label "VC2"
 		(at 27.94 127 0)
-		(fields_autoplaced yes)
 		(effects
 			(font
@@
 	(label "to_rx"
 		(at 139.7 129.54 0)
-		(fields_autoplaced yes)
 		(effects
 			(font
@@
 	(label "VC11"
 		(at 27.94 104.14 0)
-		(fields_autoplaced yes)
 		(effects
 			(font
@@
 	(label "VC13"
 		(at 85.09 91.44 0)
-		(fields_autoplaced yes)
 		(effects
 			(font
@@
 	(label "VC4"
 		(at 85.09 125.73 0)
-		(fields_autoplaced yes)
 		(effects
 			(font
@@
 	(label "CB4"
 		(at 143.51 64.77 180)
-		(fields_autoplaced yes)
 		(effects
 			(font
@@
 	(label "CB0"
 		(at 64.77 132.08 180)
-		(fields_autoplaced yes)
 		(effects
 			(font
@@
 	(label "CB9"
 		(at 143.51 52.07 180)
-		(fields_autoplaced yes)
 		(effects
 			(font
@@
 	(label "VC10"
 		(at 27.94 106.68 0)
-		(fields_autoplaced yes)
 		(effects
 			(font
@@
 	(label "VC7"
 		(at 85.09 114.3 0)
-		(fields_autoplaced yes)
 		(effects
 			(font
@@
 	(label "VC8"
 		(at 27.94 111.76 0)
-		(fields_autoplaced yes)
 		(effects
 			(font
@@
 	(label "VC1"
 		(at 27.94 129.54 0)
-		(fields_autoplaced yes)
 		(effects
 			(font
@@
 	(label "VC8"
 		(at 85.09 110.49 0)
-		(fields_autoplaced yes)
 		(effects
 			(font
@@
 	(label "CB5"
 		(at 143.51 62.23 180)
-		(fields_autoplaced yes)
 		(effects
 			(font
@@
 	(label "VC11"
 		(at 85.09 99.06 0)
-		(fields_autoplaced yes)
 		(effects
 			(font
@@
 	(label "VC1"
 		(at 85.09 137.16 0)
-		(fields_autoplaced yes)
 		(effects
 			(font
@@
 	(label "CB0"
 		(at 143.51 74.93 180)
-		(fields_autoplaced yes)
 		(effects
 			(font
@@
 	(label "CB12"
 		(at 143.51 44.45 180)
-		(fields_autoplaced yes)
 		(effects
 			(font
@@
 	(label "VC6"
 		(at 27.94 116.84 0)
-		(fields_autoplaced yes)
 		(effects
 			(font
@@
 	(label "CB10"
 		(at 143.51 49.53 180)
-		(fields_autoplaced yes)
 		(effects
 			(font
@@
 	(label "VC0"
 		(at 85.09 140.97 0)
-		(fields_autoplaced yes)
 		(effects
 			(font
@@
 	(label "VC12"
 		(at 85.09 95.25 0)
-		(fields_autoplaced yes)
 		(effects
 			(font
@@
 	(label "VC5"
 		(at 85.09 121.92 0)
-		(fields_autoplaced yes)
 		(effects
 			(font
@@
 	(label "CB12"
 		(at 64.77 101.6 180)
-		(fields_autoplaced yes)
 		(effects
 			(font
@@
 	(label "CB5"
 		(at 64.77 119.38 180)
-		(fields_autoplaced yes)
 		(effects
 			(font
@@
 	(label "CB10"
 		(at 64.77 106.68 180)
-		(fields_autoplaced yes)
 		(effects
 			(font
@@
 	(label "to_rx"
 		(at 87.63 33.02 0)
-		(fields_autoplaced yes)
 		(effects
 			(font
@@
 	(label "VC3"
 		(at 27.94 124.46 0)
-		(fields_autoplaced yes)
 		(effects
 			(font
@@
 	(label "CB13"
 		(at 64.77 99.06 180)
-		(fields_autoplaced yes)
 		(effects
 			(font
@@
 	(label "VC7"
 		(at 27.94 114.3 0)
-		(fields_autoplaced yes)
 		(effects
 			(font
@@
 	(label "CB9"
 		(at 64.77 109.22 180)
-		(fields_autoplaced yes)
 		(effects
 			(font
@@
 	(label "VC6"
 		(at 85.09 118.11 0)
-		(fields_autoplaced yes)
 		(effects
 			(font
@@
 	(label "VC13"
 		(at 27.94 99.06 0)
-		(fields_autoplaced yes)
 		(effects
 			(font
@@
 	(label "VC4"
 		(at 27.94 121.92 0)
-		(fields_autoplaced yes)
 		(effects
 			(font
@@
 	(label "CB3"
 		(at 64.77 124.46 180)
-		(fields_autoplaced yes)
 		(effects
 			(font
@@
 	(label "CB4"
 		(at 64.77 121.92 180)
-		(fields_autoplaced yes)
 		(effects
 			(font
@@
 	(label "CB7"
 		(at 64.77 114.3 180)
-		(fields_autoplaced yes)
 		(effects
 			(font
@@
 	(label "CB1"
 		(at 64.77 129.54 180)
-		(fields_autoplaced yes)
 		(effects
 			(font
@@
 	(label "VC5"
 		(at 27.94 119.38 0)
-		(fields_autoplaced yes)
 		(effects
 			(font
@@
 	(label "VC3"
 		(at 85.09 129.54 0)
-		(fields_autoplaced yes)
 		(effects
 			(font
@@
 	(label "CB2"
 		(at 64.77 127 180)
-		(fields_autoplaced yes)
 		(effects
 			(font
@@
 	(label "CB8"
 		(at 143.51 54.61 180)
-		(fields_autoplaced yes)
 		(effects
 			(font
@@
 	(label "CB3"
 		(at 143.51 67.31 180)
-		(fields_autoplaced yes)
 		(effects
 			(font
@@
 	(label "CB8"
 		(at 64.77 111.76 180)
-		(fields_autoplaced yes)
 		(effects
 			(font
@@
 	(label "CB7"
 		(at 143.51 57.15 180)
-		(fields_autoplaced yes)
 		(effects
 			(font
@@
 	(label "VC9"
 		(at 27.94 109.22 0)
-		(fields_autoplaced yes)
 		(effects
 			(font
@@
 	(label "VC9"
 		(at 85.09 106.68 0)
-		(fields_autoplaced yes)
 		(effects
 			(font
@@
 	(label "VC12"
 		(at 27.94 101.6 0)
-		(fields_autoplaced yes)
 		(effects
 			(font
@@
 	(label "CB2"
 		(at 143.51 69.85 180)
-		(fields_autoplaced yes)
 		(effects
 			(font
@@
 	(label "CB6"
 		(at 143.51 59.69 180)
-		(fields_autoplaced yes)
 		(effects
 			(font
@@
 	(label "VC2"
 		(at 85.09 133.35 0)
-		(fields_autoplaced yes)
 		(effects
 			(font
@@
 	(label "CB13"
 		(at 143.51 41.91 180)
-		(fields_autoplaced yes)
 		(effects
 			(font
@@
 		(shape input)
 		(at 137.16 113.03 0)
-		(fields_autoplaced yes)
 		(effects
 			(font
@@
 		(shape input)
 		(at 137.16 105.41 0)
-		(fields_autoplaced yes)
 		(effects
 			(font
@@
 		(shape input)
 		(at 137.16 107.95 0)
-		(fields_autoplaced yes)
 		(effects
 			(font
@@
 		(shape input)
 		(at 137.16 115.57 0)
-		(fields_autoplaced yes)
 		(effects
 			(font
@@
 			)
 		)
-		(property "Value" "300	"
+		(property "Value" "300"
 			(at 63.5 78.74 90)
 			(effects
@@
 		(at 35.56 91.44)
 		(size 20.32 43.18)
+		(exclude_from_sim no)
+		(in_bom yes)
+		(on_board yes)
+		(dnp no)
 		(fields_autoplaced yes)
 		(stroke
@@
 		(at 143.51 77.47)
 		(size 20.32 24.13)
+		(exclude_from_sim no)
+		(in_bom yes)
+		(on_board yes)
+		(dnp no)
 		(fields_autoplaced yes)
 		(stroke
