File: BMS/Temperature_LTC_1.kicad_sch (KiCad schematic)
At the start: 35 parts, among them J16 Harwin M80-8542042

Commit message: zmiany w bq79614 layout
Parts:
- removed J16: Harwin M80-8542042, footrpint:HARWIN_M80-8542042, symbol M80-8542042:M80-8542042
- added J16: Conn_01x10, footrpint:HARWIN_G125-MV11005L1P, symbol Connector_Generic:Conn_01x10
- TH1: footprint (none) -> Resistor_SMD:R_0603_1608Metric_Pad0.98x0.95mm_HandSolder; now fitted; now in the parts list
Connections:
- net GND_HV: now also J16.6 (Pin_6), J16.7 (Pin_7), J16.8 (Pin_8)
- net Thermistor2: now also J16.1 (Pin_1)
- net Thermistor3: now also J16.2 (Pin_2)
- net Thermistor4: now also J16.3 (Pin_3)
- net Thermistor5: now also J16.4 (Pin_4)
- net Thermistor6: now also J16.5 (Pin_5)
- net Thermistor7: now also J16.10 (Pin_10)
- net Thermistor8: now also J16.9 (Pin_9)
- net Thermistor1: no longer names the net of R14.2, R15.1, R8.2, TH1.1
- no-connect marks 4 -> 0

Commit message: Iteracja 1.0 gotowa, teraz sprawdzenie i zmiany kosmetyczne
Changed lines of the file:
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@@
 (kicad_sch
-	(version 20231120)
+	(version 20250114)
 	(generator "eeschema")
-	(generator_version "8.0")
+	(generator_version "9.0")
 	(paper "A4")
 	(junction
@@
 	(label "Thermistor3"
 		(at 81.28 83.82 180)
-		(fields_autoplaced yes)
 		(effects
 			(font
@@
 	(label "Thermistor6"
 		(at 81.28 91.44 180)
-		(fields_autoplaced yes)
 		(effects
 			(font
@@
 	(label "Thermistor6"
 		(at 189.23 35.56 0)
-		(fields_autoplaced yes)
 		(effects
 			(font
@@
 	(label "Thermistor5"
 		(at 128.27 154.94 0)
-		(fields_autoplaced yes)
 		(effects
 			(font
@@
 	(label "Thermistor5"
 		(at 81.28 88.9 180)
-		(fields_autoplaced yes)
 		(effects
 			(font
@@
 	(label "Thermistor8"
 		(at 189.23 96.52 0)
-		(fields_autoplaced yes)
 		(effects
 			(font
@@
 	(label "Thermistor8"
 		(at 81.28 101.6 180)
-		(fields_autoplaced yes)
 		(effects
 			(font
@@
 	(label "Thermistor3"
 		(at 129.54 97.79 0)
-		(fields_autoplaced yes)
 		(effects
 			(font
@@
 	(label "Thermistor7"
 		(at 189.23 66.04 0)
-		(fields_autoplaced yes)
 		(effects
 			(font
@@
 	(label "Thermistor4"
 		(at 81.28 86.36 180)
-		(fields_autoplaced yes)
 		(effects
 			(font
@@
 	(label "Thermistor2"
 		(at 81.28 81.28 180)
-		(fields_autoplaced yes)
 		(effects
 			(font
@@
 	(label "Thermistor4"
 		(at 128.27 123.19 0)
-		(fields_autoplaced yes)
 		(effects
 			(font
@@
 	(label "Thermistor2"
 		(at 129.54 69.85 0)
-		(fields_autoplaced yes)
 		(effects
 			(font
@@
 	(label "Thermistor7"
 		(at 81.28 104.14 180)
-		(fields_autoplaced yes)
 		(effects
 			(font
@@
 		(shape input)
 		(at 110.49 158.75 180)
-		(fields_autoplaced yes)
 		(effects
 			(font
@@
 		(shape input)
 		(at 204.47 69.85 0)
-		(fields_autoplaced yes)
 		(effects
 			(font
@@
 		(shape input)
 		(at 111.76 125.73 180)
-		(fields_autoplaced yes)
 		(effects
 			(font
@@
 		(shape input)
 		(at 204.47 100.33 0)
-		(fields_autoplaced yes)
 		(effects
 			(font
@@
 		(shape input)
 		(at 172.72 100.33 180)
-		(fields_autoplaced yes)
 		(effects
 			(font
@@
 		(shape input)
 		(at 113.03 73.66 180)
-		(fields_autoplaced yes)
 		(effects
 			(font
@@
 		(shape input)
 		(at 144.78 73.66 0)
-		(fields_autoplaced yes)
 		(effects
 			(font
@@
 		(shape input)
 		(at 113.03 100.33 180)
-		(fields_autoplaced yes)
 		(effects
 			(font
@@
 		(shape input)
 		(at 143.51 158.75 0)
-		(fields_autoplaced yes)
 		(effects
 			(font
@@
 		(shape input)
 		(at 93.98 45.72 180)
-		(fields_autoplaced yes)
 		(effects
 			(font
@@
 		(shape input)
 		(at 172.72 40.64 180)
-		(fields_autoplaced yes)
 		(effects
 			(font
@@
 		(shape input)
 		(at 204.47 40.64 0)
-		(fields_autoplaced yes)
 		(effects
 			(font
@@
 		(shape input)
 		(at 144.78 100.33 0)
-		(fields_autoplaced yes)
 		(effects
 			(font
@@
 		(shape input)
 		(at 143.51 125.73 0)
-		(fields_autoplaced yes)
 		(effects
 			(font
@@
 		(shape input)
 		(at 172.72 69.85 180)
-		(fields_autoplaced yes)
 		(effects
 			(font
@@
 		(shape input)
 		(at 116.84 30.48 180)
-		(fields_autoplaced yes)
-		(effects
-			(font
+		(effects
+			(font
