File: Hardware/Connectivity.kicad_sch (KiCad schematic)
At the start: 83 parts, among them J11 USB4235-03-C_REVA, J13 USB_A, J17 Conn_01x04, J19 Conn_02x13_Counter_Clockwise, J2 Conn_01x02, J20 Conn_01x04, J3 Conn_01x02, J4 Conn_01x02, J7 FTSH-107-01-L-D-K, J8 Conn_01x02, J9 Conn_01x02, Q3 DMT6018LDR-7, Q4 DMT6018LDR-7, Q5 DMT6018LDR-7, Q6 DMT6018LDR-7, Q7 DMT6018LDR-7, SW1 SW_Push, U4 MCP2542FD-E/MF

Commit message: Male zmiany
Parts:
- R164: value 300 -> 1k
Changed lines of the file:
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@@
 			)
 		)
-		(property "Value" "300"
+		(property "Value" "1k"
 			(at 34.29 169.9514 90)
 			(effects
