File: Hardware/Connectivity.kicad_sch (KiCad schematic)
At the start: 83 parts, among them J11 USB4235-03-C_REVA, J13 USB_A, J17 Conn_01x04, J19 Conn_02x13_Counter_Clockwise, J2 Conn_01x02, J20 Conn_01x04, J3 Conn_01x02, J4 Conn_01x02, J7 FTSH-107-01-L-D-K, J8 Conn_01x02, J9 Conn_01x02, Q3 DMT6018LDR-7, Q4 DMT6018LDR-7, Q5 DMT6018LDR-7, Q6 DMT6018LDR-7, Q7 DMT6018LDR-7, SW1 SW_Push, U4 MCP2542FD-E/MF

Commit message: Bms plug and play, 2nd iteration with the same pinout
Parts:
- removed D11: ESDA5V3SC5, Package_TO_SOT_SMD:SOT-23-5, symbol Power_Protection:ESDA5V3SC5
- removed J11: USB4235-03-C_REVA, footrpint:GCT_USB4235-03-C_REVA, symbol USB4235-03-C_REVA:USB4235-03-C_REVA
- removed J13: USB_A, footrpint:USB1046GF0190LBA, symbol Connector:USB_A
- removed JP1: Jumper_2_Small_Open, Jumper:SolderJumper-2_P1.3mm_Open_Pad1.0x1.5mm, symbol Jumper:Jumper_2_Small_Open
- removed Q3, Q4, Q6: DMT6018LDR-7, Samacsys:DMT6018LDR7, symbol Samacsys_kicad_sym:DMT6018LDR-7
- removed Q5, Q7: DMT6018LDR-7, DMT6018LDR7, symbol DMT6018LDR-7:DMT6018LDR-7
- removed R160: 100, Resistor_SMD:R_0603_1608Metric_Pad0.98x0.95mm_HandSolder, symbol Device:R_Small
- added C138, C142, C143, C144: 100nF, Capacitor_SMD:C_0603_1608Metric, symbol Device:C_Small
- added D11, D19, D8: 60V/0.5/3A, Diode_SMD:D_SOD-123, symbol Device:D_Schottky_Small
- added D15: ESDA5V3SC5, Package_TO_SOT_SMD:SOT-23-5, symbol Power_Protection:ESDA5V3SC5
- added J12, J13: TYPE-C-31-M-12, footrpint:HRO_TYPE-C-31-M-12, symbol TYPE-C-31-M-12:TYPE-C-31-M-12
- added Q1, Q3, Q4: STD3NK90ZT4, Package_TO_SOT_SMD:TO-252-2, symbol Transistor_FET_Other:Q_NMOS_Depletion_GDS
- added R101, R126: 5.1K, Resistor_SMD:R_0603_1608Metric, symbol Device:R_Small
- added R127, R128, R129, R130: 0R, Resistor_SMD:R_0603_1608Metric, symbol Device:R_Small
- added R166: 120R, Resistor_SMD:R_0603_1608Metric, symbol Device:R_Small
- added R171, R172: 10k, Resistor_SMD:R_0603_1608Metric, symbol Device:R_Small
- added R177, R178: 33, Resistor_SMD:R_0603_1608Metric, symbol Device:R_Small
- added SW2, SW3: SW_Push, footrpint:1478732, symbol Switch:SW_Push
- added U5: ESP32-C3-WROOM-02U, RF_Module:ESP32-C3-WROOM-02U, symbol RF_Module:ESP32-C3-WROOM-02U
- J5, J6: value ~ -> (none)
- R155: value 300 -> 1k
- R162: value 130 -> 1k
- R164: value 1k -> 3k
- R173, R174: value 33 -> 10k; Manufacturer_Name -- -> (none); Manufacturer_Part_Number -- -> (none); Mouser Part Number 71-CRCW060333R0FKEC -> (none)
- U4: footprint Package_DFN_QFN:DFN-8-1EP_3x3mm_P0.65mm_EP1.55x2.4mm -> footrpint:SOIC127P600X175-8N
Connections:
- net +5V_curr_sense is gone; now on net +5V: C115.2, D6.1 (K), J17.4 (Pin_4), J19.2 (Pin_2)
- net Curr_sense_out is gone; now on net Curr_sense: J17.3 (Pin_3), J19.18 (Pin_18), TP4.1
- net USB2 - is gone; now on net GND: R174.1
- net +12V: now also D8.1 (K)
- net +3.3V: now also R173.2, C138.2, C142.2, C143.2, R172.2, U5.1 (3V3)
- net 5V_fused_minus: now also D8.2 (A), Q4.2 (D)
- net B2_IN: no longer J2.1 (Pin_1)
- net B3_IN: no longer J3.1 (Pin_1)
- net B4_IN: no longer J4.1 (Pin_1)
- net D1: now also Q1.2 (D)
- net D2: now also Q3.2 (D)
- net EX_CANFD+: now also D7.4 (K), R166.2; no longer D7.5 (K)
- net EX_CANFD-: now also D7.5 (K), R166.1; no longer D7.4 (K)
- net G1: now also Q1.1 (G)
- net G2: now also Q3.1 (G)
- net G3: now also Q4.1 (G)
- net GND: now also C138.1, C142.1, C143.1, C144.1, D15.2 (A), J12.A1_B12 (GND), J12.B1_A12 (GND), J13.A1_B12 (GND), J13.B1_A12 (GND), Q1.3 (S), Q3.3 (S), Q4.3 (S), R101.2, R126.1, R171.1, SW2.1, SW3.1, U5.19 (GND), U5.9 (GND); no longer J2.2 (Pin_2), J3.2 (Pin_2), J4.2 (Pin_2), U4.9 (VSS)
- net USB1_DN: now also D12.3 (K), D12.4 (K), J12.A7 (DN1), J12.B7 (DN2); no longer D12.1 (K), D12.5 (K)
- net USB1_DP: now also D12.1 (K), D12.5 (K), J12.A6 (DP1), J12.B6 (DP2); no longer D12.3 (K), D12.4 (K)
- net VBUS: now also D11.2 (A), D19.2 (A), J12.A4_B9 (VBUS), J12.B4_A9 (VBUS), J13.A4_B9 (VBUS), J13.B4_A9 (VBUS)
- net at R174.2: now also J12.S1 (SHIELD), J12.S2 (SHIELD), J12.S3 (SHIELD), J12.S4 (SHIELD)
- net at R76.1: now also J12.A5 (CC1)
- net at R75.2: now also J12.B5 (CC2)
- net USB2 + renamed Program_esp
- net Program_esp: now also C144.2, SW3.2, U5.2 (EN)
- new net: R128.2, U5.12 (IO21/TXD)
- new net: R130.1, U5.3 (IO4)
- new net: R127.2, U5.11 (IO20/RXD)
- new net: R129.1, U5.15 (IO3)
- new net: R172.1, U5.16 (IO2), U5.7 (IO8)
- new net: SW2.2, U5.8 (IO9)
- new net: J13.B5 (CC2), R126.2
- new net: J13.A5 (CC1), R101.1
- new net: J13.S1 (SHIELD), J13.S2 (SHIELD), J13.S3 (SHIELD), J13.S4 (SHIELD), R171.2
- new net 5V_USB: D11.1 (K), D19.1 (K)
- new net USB2+: R177.1, U5.14 (IO19)
- new net USB2-: R178.1, U5.13 (IO18)
- new net USB2_DN: D15.3 (K), D15.4 (K), J13.A7 (DN1), J13.B7 (DN2), R178.2
- new net USB2_DP: D15.1 (K), D15.5 (K), J13.A6 (DP1), J13.B6 (DP2), R177.2
- new net esp32_RX1: R127.1
- new net esp32_RX2: R129.2
- new net esp32_TX1: R128.1
- new net esp32_TX2: R130.2
- no-connect marks 12 -> 9
Other:
- note removed: "USB_A"
- moved on the sheet: J8
