File: Hardware/Connectivity.kicad_sch (KiCad schematic)
At the start: 100 parts, among them J12 TYPE-C-31-M-12, J13 TYPE-C-31-M-12, J17 Conn_01x04, J19 Conn_02x13_Counter_Clockwise, J2 Conn_01x02, J20 Conn_01x04, J3 Conn_01x02, J4 Conn_01x02, J7 FTSH-107-01-L-D-K, J8 Conn_01x02, J9 Conn_01x02, Q1 STD3NK90ZT4, Q3 STD3NK90ZT4, Q4 STD3NK90ZT4, SW1 SW_Push, SW2 SW_Push, SW3 SW_Push, U4 MCP2542FD-E/MF, U5 ESP32-C3-WROOM-02U

Commit message: nearly done
Parts:
- removed R127, R128: 0R, Resistor_SMD:R_0603_1608Metric, symbol Device:R_Small
- removed R166: 120R, Resistor_SMD:R_0603_1608Metric, symbol Device:R_Small
- removed TP1, TP10, TP11, TP17, TP18, TP2, TP3, TP4, TP5, TP6, TP7, TP8, TP9: TestPoint_Small, TestPoint:TestPoint_Pad_D1.0mm, symbol Connector:TestPoint_Small
- added C147, C148: 100nF, Capacitor_SMD:C_0603_1608Metric_Pad1.08x0.95mm_HandSolder, symbol Device:C_Small
- added D20: ESDA5V3SC5, Package_TO_SOT_SMD:SOT-23-5, symbol Power_Protection:ESDA5V3SC5
- added D21, D22, D23: 60V/0.5/3A, Diode_SMD:D_SOD-123, symbol Device:D_Schottky_Small
- added F47: 400mA, Fuse:Fuse_0805_2012Metric, symbol Device:Fuse_Small
- added Q5, Q6, Q7: STD3NK90ZT4, Package_TO_SOT_SMD:TO-252-2, symbol Transistor_FET_Other:Q_NMOS_Depletion_GDS
- added R131, R133, R135: 10k, Resistor_SMD:R_0603_1608Metric, symbol Device:R_Small
- added R132, R134, R62: 100, Resistor_SMD:R_0603_1608Metric, symbol Device:R_Small
- added R180, R181: 120R, Resistor_SMD:R_0603_1608Metric, symbol Device:R_Small
- added U6: MCP2542FD-E/MF, footrpint:SOIC127P600X175-8N, symbol Interface_CAN_LIN:MCP2542FDxMF
Connections:
- net +12V: now also D21.1 (K), D22.1 (K), D23.1 (K)
- net +3.3V: now also C147.2, U6.5 (VIO)
- net +5V: now also C148.1, F47.1, U6.3 (VDD); no longer J19.2 (Pin_2)
- net +5V_external: no longer J19.10 (Pin_10), J19.9 (Pin_9)
- net 5V_fused_minus: no longer J19.8 (Pin_8)
- net EX_CANFD+: now also D20.3 (K), D20.4 (K), R180.2, R181.2, U6.7 (CANH)
- net EX_CANFD-: now also D20.1 (K), D20.5 (K), R180.1, R181.1, U6.6 (CANL)
- net GND: now also C147.1, C148.2, D20.2 (A), Q5.3 (S), Q6.3 (S), Q7.3 (S), R131.1, R133.1, R135.1, U6.2 (VSS), U6.8 (STBY); no longer J19.21 (Pin_21), J19.23 (Pin_23), J19.25 (Pin_25)
- net esp32_RX1: now also U5.11 (IO20/RXD)
- net esp32_TX1: now also U5.12 (IO21/TXD)
- net relay_enable2: now reaches U5.17 (IO1)
- net relay_enable2: now also R132.1
- net relay_enable1: now reaches U5.18 (IO0)
- net relay_enable1: now also R62.1
- net esp32_can_tx: now reaches U5.5 (IO6)
- net esp32_can_tx: now also U6.1 (TXD)
- net esp32_can_rx: now reaches U5.6 (IO7)
- net esp32_can_rx: now also U6.4 (RXD)
- net G3: no longer names the net of Q4.1 (G), R161.2, R163.2
- new net: Q6.1 (G), R132.2, R133.2
- new net: Q5.1 (G), R131.2, R62.2
- new net: Q7.1 (G), R134.2, R135.2
- new net: F47.2, J19.2 (Pin_2)
- new net Relay_OUT2: D21.2 (A), J19.8 (Pin_8), Q5.2 (D)
- new net Relay_OUT3: D22.2 (A), J19.9 (Pin_9), Q6.2 (D)
- new net Relay_OUT4: D23.2 (A), J19.10 (Pin_10), Q7.2 (D)
- new net SPI_CLK: J19.21 (Pin_21)
- new net SPI_MISO: J19.25 (Pin_25)
- new net SPI_MOSI: J19.23 (Pin_23)
- new net relay_enable3: R134.1
Other:
- note removed: "DMT6018LDR-7 is a package with 2 mossfets inside."
- moved on the sheet: D15, D19, J13, R171, R178

Commit message: New connectors jst_xh for low voltage side of bms
Parts:
- removed C115, C118: 0.1u, Capacitor_SMD:C_0603_1608Metric_Pad1.08x0.95mm_HandSolder, symbol Device:C_Small
- removed D11: 60V/0.5/3A, Diode_SMD:D_SOD-123, symbol Device:D_Schottky_Small
- removed D12, D15, D20, D6, D7: ESDA5V3SC5, Package_TO_SOT_SMD:SOT-23-5, symbol Power_Protection:ESDA5V3SC5
- removed F47: 400mA, Fuse:Fuse_0805_2012Metric, symbol Device:Fuse_Small
- removed J17: Conn_01x04, footrpint:HARWIN_M80-5100442, symbol Connector_Generic:Conn_01x04
- removed J19: Conn_02x13_Counter_Clockwise, footrpint:HARWIN_M80-5002642, symbol Connector_Generic:Conn_02x13_Counter_Clockwise
- added D20: 60V/0.5/3A, Diode_SMD:D_SOD-123, symbol Device:D_Schottky_Small
- added D27, D28, D29, D30: 12V, Diode_SMD:D_SOD-323, symbol Device:D_Schottky_Small
- added D31, D32, D33, D34, D35, D36, D37: 13.3V tvs, Package_TO_SOT_SMD:SOT-23, symbol Device:D_TVS_Dual_AAC
- added F48, F49, F50, F51, F52, F6: 1A 24V, Fuse:Fuse_1206_3216Metric, symbol Device:Fuse_Small
- added F55: 400mA, Fuse:Fuse_0805_2012Metric, symbol Device:Fuse_Small
- added J17: S2B-XH-A(LF)(SN), Connector_JST:JST_XH_S2B-XH-A_1x02_P2.50mm_Horizontal, symbol Connector_Generic:Conn_01x02
- added J21: S6B-XH-A-1(LF)(SN), Connector_JST:JST_XH_S6B-XH-A_1x06_P2.50mm_Horizontal, symbol Connector_Generic:Conn_01x06
- added J22: S3B-XH-A(LF)(SN), Connector_JST:JST_XH_S3B-XH-A_1x03_P2.50mm_Horizontal, symbol Connector_Generic:Conn_01x03
- added J23: S8B-XH-A(LF)(SN), Connector_JST:JST_XH_S8B-XH-A_1x08_P2.50mm_Horizontal, symbol Connector_Generic:Conn_01x08
- added J24: S5B-XH-A(LF)(SN), Connector_JST:JST_XH_S5B-XH-A_1x05_P2.50mm_Horizontal, symbol Connector_Generic:Conn_01x05
- added R160, R185, R188, R191: 500, Resistor_SMD:R_0603_1608Metric, symbol Device:R_Small
- added R166, R183, R186, R189: 15k, Resistor_SMD:R_0603_1608Metric, symbol Device:R_Small
- added R182, R184, R187, R190: 5.6k, Resistor_SMD:R_0603_1608Metric, symbol Device:R_Small
- R171, R174: value 10k -> 1M
Connections:
- net +5V: now also F55.2
- net 12V_IN: now also J17.2 (Pin_2)
- net 5V_USB: now also D20.1 (K)
- net 5V_fused_minus: now also F6.2, J21.3 (Pin_3); no longer D8.2 (A), Q4.2 (D)
- net B2_IN: now also D31.2 (A2), J23.7 (Pin_7)
- net B3_IN: now also D32.1 (A1), J23.6 (Pin_6)
- net B4_IN: now also D33.1 (A1), J23.5 (Pin_5)
- net D1: now also F49.1; no longer J5.2 (Pin_2)
- net D2: now also F48.1; no longer J6.2 (Pin_2)
- net EX_CANFD+: now also D35.2 (A2), D37.2 (A2), J22.3 (Pin_3)
- net EX_CANFD-: now also D35.1 (A1), D37.1 (A1), J22.1 (Pin_1)
- net GND: now also D27.2 (A), D28.2 (A), D29.2 (A), D30.2 (A), D31.3 (common), D32.3 (common), D33.3 (common), D34.3 (common), D35.3 (common), D36.3 (common), D37.3 (common), J17.1 (Pin_1), J24.1 (Pin_1), R182.1, R184.1, R187.1, R190.1
- net Relay_OUT2: now also F51.2, J21.2 (Pin_2); no longer D21.2 (A), Q5.2 (D)
- net Relay_OUT3: now also F52.2, J21.1 (Pin_1); no longer D22.2 (A), Q6.2 (D)
- net Relay_OUT4: now also F50.2, J21.6 (Pin_6); no longer D23.2 (A), Q7.2 (D)
- net SPI_CLK: now also J24.3 (Pin_3)
- net SPI_MISO: now also J24.5 (Pin_5)
- net SPI_MOSI: now also J24.4 (Pin_4)
- net USB1_DN: now also D34.1 (A1)
- net USB1_DP: now also D34.2 (A2)
- net USB2_DN: now also D36.1 (A1)
- net USB2_DP: now also D36.2 (A2)
- net VBUS: no longer names the net of D19.2 (A), J13.A4_B9 (VBUS), J13.B4_A9 (VBUS)
- net VBUS: no longer J12.A4_B9 (VBUS), J12.B4_A9 (VBUS)
- new net: D20.2 (A), J12.A4_B9 (VBUS), J12.B4_A9 (VBUS)
- new net: D23.2 (A), F50.1, Q7.2 (D)
- new net: D28.1 (K), R183.2, R185.1
- new net: D30.1 (K), R189.2, R191.1
- new net: D22.2 (A), F52.1, Q6.2 (D)
- new net: D21.2 (A), F51.1, Q5.2 (D)
- new net: D27.1 (K), R160.1, R166.2
- new net: D29.1 (K), R186.2, R188.1
- new net +5V_curr_sense: F55.1, J23.8 (Pin_8), J24.2 (Pin_2)
- new net 12V_Analog_Input1: J23.4 (Pin_4), R160.2
- new net 12V_Analog_Input2: J23.3 (Pin_3), R185.2
- new net 12V_Analog_Input3: J23.2 (Pin_2), R188.2
- new net 12V_Analog_Input4: J23.1 (Pin_1), R191.2
- new net Analog_Input1: R166.1, R182.2
- new net Analog_Input2: R183.1, R184.2
- new net Analog_Input3: R186.1, R187.2
- new net Analog_Input4: R189.1, R190.2
- new net CLK: D33.2 (A2)
- new net D3: D8.2 (A), F6.1, Q4.2 (D)
- new net MISO: D31.1 (A1)
- new net MOSI: D32.2 (A2)
- new net PreCharge_OUT: F48.2, J21.5 (Pin_5), J6.2 (Pin_2)
- new net Relay_OUT: F49.2, J21.4 (Pin_4), J5.2 (Pin_2)
Other:
- note added: "ESP32"
- note removed: "Curr_sense2 jest opcjonalnym sygnałem jak"
- note removed: "Current Sensor"
- note removed: "będzie czujnik 4 pinowy"
- moved on the sheet: C138, C142, C143, C144, C147, C148, D19, D21, D22, D23, J9, Q5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

Commit message: No drc errors
Parts:
- removed D31, D32: 13.3V tvs, Package_TO_SOT_SMD:SOT-23, symbol Device:D_TVS_Dual_AAC
- added D45: 13.3V tvs, Package_TO_SOT_SMD:SOT-23, symbol Device:D_TVS_Dual_AAC
Connections:
- net CLK is gone; now on net +12V_curr_sense: D33.2 (A2)
- net +12V: now also F55.2
- net +5V: no longer F55.2
- net B4_IN: no longer D33.1 (A1)
- net GND: now also D45.3 (common)
- net SPI_CLK: now also D33.1 (A1)
- net SPI_MISO: now also D45.1 (A1)
- net SPI_MOSI: now also D45.2 (A2)
- net +5V_curr_sense renamed +12V_curr_sense
