File: Hardware/BMS.kicad_pcb (KiCad board)
At the start: 4 copper layers, 109 x 148 mm, 368 parts, among them IC1 STM32H742VIT6, IC2 TPS563200DDCR, J1 Conn_01x28, J10 Conn_01x10, J11 USB4235-03-C_REVA, J13 USB_A, J16 Conn_01x10, J19 Conn_02x13_Counter_Clockwise, J7 FTSH-107-01-L-D-K, Q2 100V/2W, Q5 DMT6018LDR-7, Q7 DMT6018LDR-7, Q8 100V/2W, SW1 SW_Push, U1 BQ79614PAPRQ1, U2 BQ79614PAPRQ1, U3 PBQ79600PWQ1, U4 MCP2542FD-E/MF, U5 PTPSM863253RDXR

Commit message: Bms plug and play, 2nd iteration with the same pinout
Parts:
- removed C12, C13, C145, C147, C61, C62: 2.2n, footrpint:CAPC5728X280N
- removed G***: LOGO, footrpint:cat4_5x5
- removed G***: LOGO, footrpint:catd3_10x10
- removed G***: LOGO, footrpint:cat2_20x20_2
- removed G***: LOGO, footrpint:cat2_15x15
- removed G***: LOGO, footrpint:cat_coffe_8x8
- removed G***: LOGO, footrpint:qr_github_12x12
- removed J11: USB4235-03-C_REVA, footrpint:GCT_USB4235-03-C_REVA
- removed JP1: Jumper_2_Small_Open, Jumper:SolderJumper-2_P1.3mm_Open_Pad1.0x1.5mm
- removed Q5, Q7: DMT6018LDR-7, Samacsys:DMT6018LDR7
- removed R131, R132, R133, R134, R135, R136, R137, R138, R139: 10, footrpint:RESC6331X80N
- removed R140, R15: 100k, Resistor_SMD:R_0603_1608Metric_Pad0.98x0.95mm_HandSolder
- removed R141, R142, R62: 10k, Resistor_SMD:R_0603_1608Metric_Pad0.98x0.95mm_HandSolder
- removed R160: 100, Resistor_SMD:R_0603_1608Metric_Pad0.98x0.95mm_HandSolder
- removed R61: 15.8k, Resistor_SMD:R_0603_1608Metric_Pad0.98x0.95mm_HandSolder
- removed TP15, TP16: TestPoint_Small, TestPoint:TestPoint_Pad_D1.0mm
- added C149: 220p, Capacitor_SMD:C_0603_1608Metric_Pad1.08x0.95mm_HandSolder, F.Cu at (208.9, 144.2)
- added C150: 220p, Capacitor_SMD:C_0603_1608Metric_Pad1.08x0.95mm_HandSolder, F.Cu at (151.4, 137.9)
- added C151: 220p, Capacitor_SMD:C_0603_1608Metric_Pad1.08x0.95mm_HandSolder, F.Cu at (151.4, 140.4)
- added C152: 220p, Capacitor_SMD:C_0603_1608Metric_Pad1.08x0.95mm_HandSolder, F.Cu at (209.2, 163.7)
- added C153: 220p, Capacitor_SMD:C_0603_1608Metric_Pad1.08x0.95mm_HandSolder, F.Cu at (281.8, 225.3)
- added D15: ESDA5V3SC5, Package_TO_SOT_SMD:SOT-23-5, F.Cu at (244.9, 186.2)
- added D19: 60V/0.5/3A, Diode_SMD:D_SOD-123, F.Cu at (239.7, 182.2)
- added F1: 400mA, Fuse:Fuse_0805_2012Metric, F.Cu at (148.7, 185.4)
- added F10: 400mA, Fuse:Fuse_0805_2012Metric, F.Cu at (148.7, 190.4)
- added F11: 400mA, Fuse:Fuse_0805_2012Metric, F.Cu at (145.2, 191.7)
- added F12: 400mA, Fuse:Fuse_0805_2012Metric, F.Cu at (148.7, 192.9)
- added F13: 400mA, Fuse:Fuse_0805_2012Metric, F.Cu at (145.2, 194.2)
- added F14: 400mA, Fuse:Fuse_0805_2012Metric, F.Cu at (148.7, 195.4)
- added F15: 400mA, Fuse:Fuse_0805_2012Metric, F.Cu at (145.2, 196.7)
- added F16: 400mA, Fuse:Fuse_0805_2012Metric, F.Cu at (148.7, 197.9)
- added F17: 400mA, Fuse:Fuse_0805_2012Metric, F.Cu at (145.2, 199.2)
- added F18: 400mA, Fuse:Fuse_0805_2012Metric, F.Cu at (148.8, 200.4)
- added F19: 400mA, Fuse:Fuse_0805_2012Metric, F.Cu at (145.2, 201.7)
- added F20: 400mA, Fuse:Fuse_0805_2012Metric, F.Cu at (148.7, 202.9)
- added F21: 400mA, Fuse:Fuse_0805_2012Metric, F.Cu at (145.2, 184.2)
- added F22: 400mA, Fuse:Fuse_0805_2012Metric, F.Cu at (65.1, 135.6)
- added F23: 400mA, Fuse:Fuse_0805_2012Metric, F.Cu at (65.1, 138.6)
- added F24: 400mA, Fuse:Fuse_0805_2012Metric, F.Cu at (65.1, 141.5)
- added F25: 400mA, Fuse:Fuse_0805_2012Metric, F.Cu at (65.1, 144.5)
- added F26: 400mA, Fuse:Fuse_0805_2012Metric, F.Cu at (69.5, 135.6)
- added F27: 400mA, Fuse:Fuse_0805_2012Metric, F.Cu at (69.5, 138.6)
- added F28: 400mA, Fuse:Fuse_0805_2012Metric, F.Cu at (69.5, 141.5)
- added F29: 400mA, Fuse:Fuse_0805_2012Metric, F.Cu at (69.5, 144.5)
- added F30: 400mA, Fuse:Fuse_0805_2012Metric, F.Cu at (73.9, 135.6)
- added F31: 400mA, Fuse:Fuse_0805_2012Metric, F.Cu at (73.9, 138.6)
- added F32: 400mA, Fuse:Fuse_0805_2012Metric, F.Cu at (73.9, 141.5)
- added F33: 400mA, Fuse:Fuse_0805_2012Metric, F.Cu at (73.9, 144.5)
- added F34: 400mA, Fuse:Fuse_0805_2012Metric, F.Cu at (78.3, 135.6)
- added F35: 400mA, Fuse:Fuse_0805_2012Metric, F.Cu at (78.3, 138.6)
- added F36: 400mA, Fuse:Fuse_0805_2012Metric, F.Cu at (78.3, 141.5)
- added F37: 400mA, Fuse:Fuse_0805_2012Metric, F.Cu at (78.3, 144.5)
- added F38: 1A, Fuse:Fuse_1206_3216Metric, F.Cu at (233.4, 183.9)
- added F39: 1A, Fuse:Fuse_1206_3216Metric, F.Cu at (216.4, 131.8)
- added F40: 400mA, Fuse:Fuse_0805_2012Metric, F.Cu at (102.1, 114.0)
- added F41: 400mA, Fuse:Fuse_0805_2012Metric, F.Cu at (102.1, 117.0)
- added F42: 400mA, Fuse:Fuse_0805_2012Metric, F.Cu at (102.1, 138.5)
- added F43: 400mA, Fuse:Fuse_0805_2012Metric, F.Cu at (102.1, 141.4)
- added F44: 400mA, Fuse:Fuse_0805_2012Metric, F.Cu at (102.1, 144.4)
- added F7: 400mA, Fuse:Fuse_0805_2012Metric, F.Cu at (145.2, 186.7)
- added F8: 400mA, Fuse:Fuse_0805_2012Metric, F.Cu at (148.7, 187.9)
- added F9: 400mA, Fuse:Fuse_0805_2012Metric, F.Cu at (145.2, 189.2)
- added IC3: TPS563200DDCR, Package_TO_SOT_SMD:SOT-23-6, F.Cu at (219.9, 136.0)
- added J12: TYPE-C-31-M-12, footrpint:HRO_TYPE-C-31-M-12, F.Cu at (253.3, 176.4)
- added L2: 3.3u 20mOhm, footrpint:CLF7045__, F.Cu at (229.1, 135.3)
- added Q1: STD3NK90ZT4, Package_TO_SOT_SMD:TO-252-2, F.Cu at (246.2, 120.0)
- added Q3: STD3NK90ZT4, Package_TO_SOT_SMD:TO-252-2, F.Cu at (246.2, 128.2)
- added Q4: STD3NK90ZT4, Package_TO_SOT_SMD:TO-252-2, F.Cu at (246.2, 135.4)
- added R167: 30K, Resistor_SMD:R_0603_1608Metric, F.Cu at (220.4, 139.5)
- added R168: 10k, Resistor_SMD:R_0603_1608Metric, F.Cu at (222.6, 138.8)
- added R169: 10k, Resistor_SMD:R_0603_1608Metric, F.Cu at (222.5, 124.0)
- added R170: 100, Resistor_SMD:R_0603_1608Metric_Pad0.98x0.95mm_HandSolder, F.Cu at (224.3, 166.4)
- added R171: 10k, Resistor_SMD:R_0603_1608Metric, F.Cu at (245.7, 191.2)
- added R172: 10k, Resistor_SMD:R_0603_1608Metric, F.Cu at (231.7, 203.9)
- added R177: 33, Resistor_SMD:R_0603_1608Metric, F.Cu at (241.2, 185.4)
- added R178: 33, Resistor_SMD:R_0603_1608Metric, F.Cu at (241.2, 186.9)
- added R179: 100, Resistor_SMD:R_0603_1608Metric_Pad0.98x0.95mm_HandSolder, F.Cu at (224.5, 161.2)
- added R77: 20R 2W, Resistor_SMD:R_2512_6332Metric, F.Cu at (45.5, 112.0)
- added R78: 20R 2W, Resistor_SMD:R_2512_6332Metric, F.Cu at (45.5, 116.9)
- added R79: 20R 2W, Resistor_SMD:R_2512_6332Metric, F.Cu at (45.5, 121.9)
- added R80: 20R 2W, Resistor_SMD:R_2512_6332Metric, F.Cu at (45.5, 126.8)
- added R81: 20R 2W, Resistor_SMD:R_2512_6332Metric, F.Cu at (45.5, 131.7)
- added R82: 20R 2W, Resistor_SMD:R_2512_6332Metric, F.Cu at (54.2, 112.0)
- added R83: 20R 2W, Resistor_SMD:R_2512_6332Metric, F.Cu at (54.2, 116.9)
- added R84: 20R 2W, Resistor_SMD:R_2512_6332Metric, F.Cu at (54.2, 121.9)
- added R85: 20R 2W, Resistor_SMD:R_2512_6332Metric, F.Cu at (54.2, 126.8)
- added R86: 20R 2W, Resistor_SMD:R_2512_6332Metric, F.Cu at (54.2, 131.7)
- added R87: 20R 2W, Resistor_SMD:R_2512_6332Metric, F.Cu at (62.9, 112.0)
- added R88: 20R 2W, Resistor_SMD:R_2512_6332Metric, F.Cu at (62.9, 116.9)
- added R89: 20R 2W, Resistor_SMD:R_2512_6332Metric, F.Cu at (62.9, 121.9)
- added R90: 20R 2W, Resistor_SMD:R_2512_6332Metric, F.Cu at (62.9, 126.8)
- added R91: 0R, Resistor_SMD:R_0603_1608Metric, F.Cu at (67.6, 172.5)
- added R92: 0R, Resistor_SMD:R_0603_1608Metric, F.Cu at (67.6, 175.0)
- added R93: 0R, Resistor_SMD:R_0603_1608Metric, F.Cu at (67.6, 177.5)
- added R94: 0R, Resistor_SMD:R_0603_1608Metric, F.Cu at (228.4, 157.4)
- added SW2: SW_Push, footrpint:1478732, F.Cu at (228.7, 181.5)
- added SW3: SW_Push, footrpint:1478732, F.Cu at (228.7, 191.3)
- added T3: SM91502ALE, footrpint:SOP254P927X572-6N, F.Cu at (224.6, 86.1)
- added T4: SM91502ALE, footrpint:SOP254P927X572-6N, F.Cu at (208.9, 136.8)
- added T5: SM91502ALE, footrpint:SOP254P927X572-6N, F.Cu at (139.0, 141.4)
- added T6: SM91502ALE, footrpint:SOP254P927X572-6N, F.Cu at (139.0, 150.8)
- added T7: SM91502ALE, footrpint:SOP254P927X572-6N, F.Cu at (209.2, 171.3)
- added T8: SM91502ALE, footrpint:SOP254P927X572-6N, F.Cu at (269.4, 235.7)
- C126: value 10uF -> 10u; footprint Capacitor_SMD:C_0603_1608Metric_Pad1.08x0.95mm_HandSolder -> Capacitor_SMD:C_0805_2012Metric_Pad1.18x1.45mm_HandSolder
- C127: value 100nF -> 10uf; footprint Capacitor_SMD:C_0603_1608Metric_Pad1.08x0.95mm_HandSolder -> Capacitor_SMD:C_0805_2012Metric_Pad1.18x1.45mm_HandSolder
- C128: value 10uF -> 100n 280mOhm; footprint Capacitor_SMD:C_0603_1608Metric_Pad1.08x0.95mm_HandSolder -> Capacitor_SMD:C_0805_2012Metric_Pad1.18x1.45mm_HandSolder
- C130, C131: value 2.2n -> 22u; footprint footrpint:CAPC5728X280N -> Capacitor_SMD:C_0603_1608Metric_Pad1.08x0.95mm_HandSolder
- C138: value 1uF -> 100nF; footprint Capacitor_SMD:C_0603_1608Metric_Pad1.08x0.95mm_HandSolder -> Capacitor_SMD:C_0603_1608Metric
- C142, C143, C144: value 2.2n -> 100nF; footprint footrpint:CAPC5728X280N -> Capacitor_SMD:C_0603_1608Metric
- C146: value 2.2n -> 220p; footprint footrpint:CAPC5728X280N -> Capacitor_SMD:C_0603_1608Metric_Pad1.08x0.95mm_HandSolder
- C65, C67, C68, C69, C70: value 1uF -> 100n
- D11: value ESDA5V3SC5 -> 60V/0.5/3A; footprint Package_TO_SOT_SMD:SOT-23-5 -> Diode_SMD:D_SOD-123
- F2, F3, F5: footprint Fuse:Fuse_0603_1608Metric_Pad1.05x0.95mm_HandSolder -> Fuse:Fuse_1206_3216Metric
- F4: value 5V/0.5A -> 400mA
- F6: value 2A -> 1A; footprint Fuse:Fuse_0603_1608Metric_Pad1.05x0.95mm_HandSolder -> Fuse:Fuse_1206_3216Metric
- IC2: footprint footrpint:TPS563200DDCR -> Package_TO_SOT_SMD:SOT-23-6
- J13: value USB_A -> TYPE-C-31-M-12; footprint footrpint:USB1046GF0190LBA -> footrpint:HRO_TYPE-C-31-M-12
- R101: value 100k -> 5.1K; footprint Resistor_SMD:R_0603_1608Metric_Pad0.98x0.95mm_HandSolder -> Resistor_SMD:R_0603_1608Metric
- R126: value 10 -> 5.1K; footprint footrpint:RESC6331X80N -> Resistor_SMD:R_0603_1608Metric
- R127, R128, R129, R130: value 10 -> 0R; footprint footrpint:RESC6331X80N -> Resistor_SMD:R_0603_1608Metric
- R155: value 300 -> 1k
- R162: value 130 -> 1k
- R164: value 1k -> 3k
- R166: value 10k 50mW -> 120R; footprint Resistor_SMD:R_0603_1608Metric_Pad0.98x0.95mm_HandSolder -> Resistor_SMD:R_0603_1608Metric
- R173, R174: value 33 -> 10k
- R33, R34, R35, R36, R37, R38, R39, R40, R41, R42, R43, R44, R45, R46: value 10 -> 20R 2W; footprint footrpint:RESC6331X80N -> Resistor_SMD:R_2512_6332Metric
- TP1, TP10, TP11, TP12, TP13, TP14, TP17, TP18, TP3, TP4, TP5, TP6, TP7, TP8, TP9: moved to F.Cu
- U1, U2: footprint footrpint:BQ79614PAPRQ1 -> Package_QFP:Texas_TQFP-64-1EP_10x10mm_P0.5mm_EP8x8mm_Mask4.44x4.44mm_ThermalVias
- U4: footprint Package_DFN_QFN:DFN-8-1EP_3x3mm_P0.65mm_EP1.55x2.4mm -> footrpint:SOIC127P600X175-8N
- U5: value PTPSM863253RDXR -> ESP32-C3-WROOM-02U; footprint footrpint:RDX0007A-MFG_NOVIA -> RF_Module:ESP32-C3-WROOM-02U
- moved TP3 235.0 mm to (388.8, 132.2)
- moved TP11 224.8 mm to (394.9, 126.2)
- moved TP10 220.9 mm to (391.9, 138.3)
- moved R46 212.5 mm to (240.7, 259.4), turned to 180 degrees
- moved R33 205.2 mm to (124.8, 244.9), turned to 90 degrees
- moved R34 201.1 mm to (129.7, 244.9), turned to 90 degrees
- moved TP18 199.5 mm to (372.9, 139.8)
- moved R35 197.2 mm to (134.7, 244.9), turned to 90 degrees
- moved TP17 195.0 mm to (372.9, 136.7)
- moved TP1 194.2 mm to (366.8, 133.7)
- moved R36 193.5 mm to (139.6, 244.9), turned to 90 degrees
- moved TP2 191.8 mm to (357.6, 110.2)
- moved R37 189.9 mm to (144.5, 244.9), turned to 90 degrees
- moved C16 182.8 mm to (84.0, 224.0)
- moved R127 178.8 mm to (248.4, 209.2)
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Connections:
- net /STM Comunication Interface /COMHN renamed /STM Comunication Interface/COMHN
- net /STM Comunication Interface /COMHP renamed /STM Comunication Interface/COMHP
- net /STM Comunication Interface /COMLN renamed /STM Comunication Interface/COMLN
- net /STM Comunication Interface /COMLP renamed /STM Comunication Interface/COMLP
- C113 pad 1: Batt_Coupling -> GND_HV2
- C115 pad 2: /Connectivity/+5V_curr_sense -> +5V
- C121 pad 1: Net-(IC2-SW) -> Net-(IC2-VBST)
- C121 pad 2: Net-(IC2-VBST) -> Net-(IC2-EN)
- C124 pad 1: /Power/5V/F_U5V -> 5V_USB
- C125 pad 2: /Power/5V/F_U5V -> 5V_USB
- C126 pad 1: +5V -> Net-(IC3-GND)
- C127 pad 1: +5V -> Net-(IC3-GND)
- C128 pad 1: Net-(U5-EN) -> Net-(IC3-VBST)
- C128 pad 2: GND -> Net-(IC3-EN)
- C129 pad 1: Batt_Coupling -> GND_HV2
- C130 pad 1: /galvanic_isulation_1/S2+ -> /Power/Power_3.3V/3.3V_unfused
- C130 pad 2: /galvanic_isulation_1/S1+ -> GND
- C131 pad 1: /galvanic_isulation_1/S2- -> /Power/Power_3.3V/3.3V_unfused
- C131 pad 2: /galvanic_isulation_1/S1- -> GND
- C132 pad 1: Stack- -> GND_HV
- C133 pad 1: Stack- -> GND_HV
- C137 pad 1: Net-(U5-FB) -> /Power/Power_3.3V/3.3V_unfused
- C138 pad 1: Net-(U5-FB) -> GND
- C138 pad 2: GND -> +3.3V
- C14 pad 1: Batt_Coupling -> GND_HV2
- C140 pad 1: Net-(C140-Pad1) -> GND
- C142 pad 1: /galvanic_isulation_1/S3+ -> GND
- C142 pad 2: /galvanic_isulation_1/S2+ -> +3.3V
- C143 pad 1: /galvanic_isulation_1/S3- -> GND
- C143 pad 2: /galvanic_isulation_1/S2- -> +3.3V
- C144 pad 1: /galvanic_isulation_2/S3- -> GND
- C144 pad 2: /galvanic_isulation_2/S2- -> /Connectivity/Program_esp
- C146 pad 1: /galvanic_isulation_0/S3- -> Net-(T3-SEC_2)
- C146 pad 2: /galvanic_isulation_0/S2- -> GND_HV
- C15 pad 1: Batt_Coupling -> GND_HV2
- C2 pad 1: Stack- -> GND_HV
- C3 pad 1: Stack- -> GND_HV
- C4 pad 1: Stack- -> GND_HV
- C42 pad 2: Stack- -> GND_HV
- C43 pad 2: Stack- -> GND_HV
- C44 pad 2: Stack- -> GND_HV
- C45 pad 2: Stack- -> GND_HV
- C46 pad 2: Stack- -> GND_HV
- C47 pad 2: Stack- -> GND_HV
- C48 pad 2: Stack- -> GND_HV
- C49 pad 2: Stack- -> GND_HV
- C5 pad 1: Stack- -> GND_HV
- C50 pad 2: Stack- -> GND_HV
- C51 pad 1: Batt_Coupling -> GND_HV2
- C52 pad 1: Batt_Coupling -> GND_HV2
- C53 pad 1: Batt_Coupling -> GND_HV2
- C54 pad 1: Batt_Coupling -> GND_HV2
- C55 pad 1: Batt_Coupling -> GND_HV2
- C56 pad 1: Batt_Coupling -> GND_HV2
- C57 pad 1: Batt_Coupling -> GND_HV2
- C58 pad 1: Batt_Coupling -> GND_HV2
- C59 pad 1: Stack- -> GND_HV
- C6 pad 1: Stack- -> GND_HV
- C60 pad 1: Stack- -> GND_HV
- C69 pad 1: GND -> +3.3V
- C69 pad 2: +3.3V -> GND
- C7 pad 1: Stack- -> GND_HV
- C71 pad 2: Batt_Coupling -> GND_HV2
- C72 pad 2: Batt_Coupling -> GND_HV2
- C73 pad 2: Batt_Coupling -> GND_HV2
- C74 pad 2: Batt_Coupling -> GND_HV2
- C75 pad 2: Batt_Coupling -> GND_HV2
- C76 pad 2: Batt_Coupling -> GND_HV2
- C77 pad 2: Batt_Coupling -> GND_HV2
- C78 pad 2: Batt_Coupling -> GND_HV2
- C79 pad 2: Batt_Coupling -> GND_HV2
- C8 pad 1: Stack- -> GND_HV
- C9 pad 1: Stack- -> GND_HV
- D11 pad 1: Net-(J13-D-) -> 5V_USB
- D11 pad 2: GND -> VBUS
- D12 pad 1: /Connectivity/USB1_DN -> /Connectivity/USB1_DP
- D12 pad 3: /Connectivity/USB1_DP -> /Connectivity/USB1_DN
- D12 pad 4: /Connectivity/USB1_DP -> /Connectivity/USB1_DN
- D12 pad 5: /Connectivity/USB1_DN -> /Connectivity/USB1_DP
- D6 pad 1: /Connectivity/+5V_curr_sense -> +5V
- D7 pad 4: /Connectivity/EX_CANFD- -> /Connectivity/EX_CANFD+
- D7 pad 5: /Connectivity/EX_CANFD+ -> /Connectivity/EX_CANFD-
- D8 pad 1: /Power/5V/F_U5V -> +12V
- D8 pad 2: VBUS -> /Connectivity/5V_fused_minus
- D9 pad 1: /Power/5V/F_U5V -> 5V_USB
- F4 pad 1: /Power/5V/F_U5V -> Net-(J16-Pin_6)
- F4 pad 2: /Power/5V/5V_unfused -> GND_HV
- F5 pad 1: Net-(U5-FB) -> /Power/Power_3.3V/3.3V_unfused
- IC1 pad 14: /NRST -> Net-(IC1-NRST)
- IC1 pad 32: /Curr_sense -> Net-(IC1-PC4)
- IC1 pad 35: /Curr_sense2 -> Net-(IC1-PB1)
- IC1 pad 51: unconnected-(IC1-PB12-Pad51) -> /UART2_RX
- IC1 pad 52: unconnected-(IC1-PB13-Pad52) -> /UART2_TX
- IC2 pad 1: GND -> +12V
- IC2 pad 2: Net-(IC2-SW) -> +12V
- IC2 pad 3: +12V -> GND
- IC2 pad 5: +12V -> Net-(IC2-EN)
- J10 pad 6: Batt_Coupling -> Net-(J10-Pin_6)
- J10 pad 7: Batt_Coupling -> Net-(J10-Pin_7)
- J10 pad 8: Batt_Coupling -> Net-(J10-Pin_8)
- J16 pad 6: Stack- -> Net-(J16-Pin_6)
- J16 pad 7: Stack- -> Net-(J16-Pin_7)
- J16 pad 8: Stack- -> Net-(J16-Pin_8)
- J19 pad 18: /Connectivity/Curr_sense_out -> /Curr_sense
- J19 pad 2: /Connectivity/+5V_curr_sense -> +5V
- L1 pad 1: Net-(IC2-SW) -> Net-(IC2-VBST)
- R101 pad 1: /Mesurements_LTC2/Temperature_LTC_2/Thermistor1 -> Net-(J13-CC1)
- R101 pad 2: Batt_Coupling -> GND
- R112 pad 1: Batt_Coupling -> Net-(F37-Pad2)
- R113 pad 1: CELL26 -> Net-(F24-Pad2)
- R114 pad 1: CELL25 -> Net-(F25-Pad2)
- R115 pad 1: CELL24 -> Net-(F26-Pad2)
- R116 pad 1: CELL23 -> Net-(F27-Pad2)
- R117 pad 1: CELL22 -> Net-(F28-Pad2)
- R118 pad 1: CELL21 -> Net-(F29-Pad2)
- R119 pad 1: CELL20 -> Net-(F30-Pad2)
- R120 pad 1: CELL19 -> Net-(F31-Pad2)
- R121 pad 1: CELL18 -> Net-(F32-Pad2)
- R122 pad 1: CELL17 -> Net-(F33-Pad2)
- R123 pad 1: CELL16 -> Net-(F34-Pad2)
- R124 pad 1: CELL15 -> Net-(F35-Pad2)
- R125 pad 1: CELL14 -> Net-(F36-Pad2)
- R126 pad 1: CELL26 -> GND
- R126 pad 2: /Mesurements_LTC2/CB13 -> Net-(J13-CC2)
- R127 pad 1: CELL25 -> /UART2_TX
- R127 pad 2: /Mesurements_LTC2/CB12 -> Net-(U5-IO20/RXD)
- R128 pad 1: CELL24 -> /UART2_RX
- R128 pad 2: /Mesurements_LTC2/CB11 -> Net-(U5-IO21/TXD)
- R129 pad 1: CELL23 -> Net-(U5-IO3)
- R129 pad 2: /Mesurements_LTC2/CB10 -> /esp32_RX2
- R130 pad 1: CELL22 -> Net-(U5-IO4)
- R130 pad 2: /Mesurements_LTC2/CB9 -> /esp32_TX2
- R166 pad 1: GND -> /Connectivity/EX_CANFD-
- R166 pad 2: Net-(IC2-VFB) -> /Connectivity/EX_CANFD+
- R173 pad 1: /USB2+ -> /Connectivity/Program_esp
- R173 pad 2: Net-(J13-D+) -> +3.3V
- R174 pad 1: /USB2- -> GND
- R174 pad 2: Net-(J13-D-) -> Net-(J12-SHIELD-PadS1)
- R19 pad 1: Stack- -> Net-(F19-Pad2)
- R2 pad 1: Batt_Coupling -> /Mesurements_LTC1/Battery/Batt1_+
- R20 pad 1: Batt_Coupling -> Net-(F1-Pad2)
- R21 pad 1: Net-(J1-Pin_13) -> Net-(F7-Pad2)
- R22 pad 1: Net-(J1-Pin_12) -> Net-(F8-Pad2)
- R23 pad 1: Net-(J1-Pin_11) -> Net-(F9-Pad2)
- R24 pad 1: Net-(J1-Pin_10) -> Net-(F10-Pad2)
- R25 pad 1: Net-(J1-Pin_9) -> Net-(F11-Pad2)
- R26 pad 1: Net-(J1-Pin_8) -> Net-(F12-Pad2)
- R27 pad 1: Net-(J1-Pin_7) -> Net-(F13-Pad2)
- R28 pad 1: Net-(J1-Pin_6) -> Net-(F14-Pad2)
- R29 pad 1: Net-(J1-Pin_5) -> Net-(F15-Pad2)
- R30 pad 1: Net-(J1-Pin_4) -> Net-(F16-Pad2)
- R31 pad 1: Net-(J1-Pin_3) -> Net-(F17-Pad2)
- R32 pad 1: Net-(J1-Pin_2) -> Net-(F18-Pad2)
- R33 pad 1: Batt_Coupling -> Net-(F1-Pad2)
- R34 pad 1: Net-(J1-Pin_13) -> Net-(F7-Pad2)
- R35 pad 1: Net-(J1-Pin_12) -> Net-(F8-Pad2)
- R36 pad 1: Net-(J1-Pin_11) -> Net-(F9-Pad2)
- R37 pad 1: Net-(J1-Pin_10) -> Net-(F10-Pad2)
- R38 pad 1: Net-(J1-Pin_9) -> Net-(F11-Pad2)
- R39 pad 1: Net-(J1-Pin_8) -> Net-(F12-Pad2)
- R4 pad 1: Batt_Coupling -> /Mesurements_LTC1/Battery/Batt1_+
- R40 pad 1: Net-(J1-Pin_7) -> Net-(F13-Pad2)
- R41 pad 1: Net-(J1-Pin_6) -> Net-(F14-Pad2)
- R42 pad 1: Net-(J1-Pin_5) -> Net-(F15-Pad2)
- R43 pad 1: Net-(J1-Pin_4) -> Net-(F16-Pad2)
- R44 pad 1: Net-(J1-Pin_3) -> Net-(F17-Pad2)
- R45 pad 1: Net-(J1-Pin_2) -> Net-(F18-Pad2)
- R46 pad 1: Stack- -> Net-(F19-Pad2)
- R64 pad 1: CELL26 -> /Mesurements_LTC2/Battery2/Batt2_+
- R66 pad 1: CELL26 -> /Mesurements_LTC2/Battery2/Batt2_+
- TH1 pad 2: Stack- -> GND_HV
- TH13 pad 2: Batt_Coupling -> GND_HV2
- TP4 pad 1: /Connectivity/Curr_sense_out -> /Curr_sense
- U1 pad 36: Stack- -> GND_HV
- U1 pad 39: Stack- -> GND_HV
- U1 pad 46: Stack- -> GND_HV
- U1 pad 50: Stack- -> GND_HV
- U1 pad 65: Stack- -> GND_HV
- U2 pad 36: Batt_Coupling -> GND_HV2
- U2 pad 39: Batt_Coupling -> GND_HV2
- U2 pad 46: Batt_Coupling -> GND_HV2
- U2 pad 50: Batt_Coupling -> GND_HV2
- U2 pad 65: Batt_Coupling -> GND_HV2
- U3 pad 2: /NFAULT -> /STM Comunication Interface/NFAULT
- U3 pad 4: /RX_1 -> /esp32_TX2
- U3 pad 5: /TX_1 -> /esp32_RX2
- U5 pad 1: +5V -> +3.3V
- U5 pad 2: unconnected-(U5-SW-Pad2) -> /Connectivity/Program_esp
- U5 pad 3: Net-(U5-FB) -> Net-(U5-IO4)
- U5 pad 4: GND -> unconnected-(U5-IO5-Pad4)
- U5 pad 6: Net-(U5-EN) -> unconnected-(U5-IO7-Pad6)
- U5 pad 7: Net-(U5-FB) -> Net-(U5-IO2)
Routing:
- net Batt_Coupling: track 303.8 -> 0.00 mm, vias 94 -> 0
- net +3.3V: track 272.4 -> 56.1 mm, vias 15 -> 4
- net +5V: track 198.5 -> 13.8 mm, vias 10 -> 0
- net /galvanic_isulation_0/S2+: track 128.3 -> 0.00 mm
- net /galvanic_isulation_0/S2-: track 126.9 -> 0.00 mm
- net /Curr_sense2: track 92.5 -> 1.65 mm, vias 3 -> 0
- net /12V_Enable: track 88.0 -> 0.00 mm, vias 2 -> 0
- net VBUS: track 118.5 -> 31.9 mm, vias 2 -> 0
- net CELL14: track 85.4 -> 0.00 mm
- net Net-(J1-Pin_13): track 81.1 -> 0.00 mm
- net CELL15: track 78.3 -> 0.00 mm
- net Net-(J1-Pin_12): track 73.5 -> 0.00 mm
- net CELL26: track 73.2 -> 0.00 mm, vias 2 -> 0
- net CELL16: track 70.6 -> 0.00 mm
- net +12V: track 76.2 -> 7.03 mm, vias 4 -> 0
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- removed copper zone on B.Cu, net +12V
- removed copper zone on F.Cu, net +12V
- removed copper zone on F.Cu, net +3.3V
- removed copper zone on F.Cu, net +5V
- removed copper zone on F.Cu, net +5V_external
- removed copper zone on F.Cu, net /Connectivity/5V_fused_minus
- removed copper zone on F.Cu, net /Power/5V/5V_unfused
- removed copper zone on F.Cu, net 12V_IN
- removed copper zone on F.Cu, net Batt_Coupling
- removed copper zone on In1.Cu, net Batt_Coupling
- removed copper zone on In2.Cu, net Batt_Coupling
- removed copper zone on B.Cu, net GND
- removed copper zone on F.Cu, net GND
- removed copper zone on In1.Cu, net GND
- removed copper zone on In2.Cu, net GND
- removed copper zone on B.Cu, net Net-(IC2-SW)
- removed copper zone on F.Cu, net Net-(IC2-SW)
- removed copper zone on F.Cu, net Stack-
- removed copper zone on In1.Cu, net Stack-
- removed copper zone on In2.Cu, net Stack-
Other:
- board size 109 x 148 mm -> 8.5 x 2 mm
- board text removed: "12V"
- board text removed: "3.3V"
- board text removed: "5V"
- board text removed: "B0"
- board text removed: "B0 is ground for BQ79614-1 and B13 is ground for BQ79614-2"
- board text removed: "B1"
- board text removed: "B10"
- board text removed: "B11"
- board text removed: "B12"
- board text removed: "B13"
- board text removed: "B14"
- board text removed: "B15"
- board text removed: "B16"
- board text removed: "B17"
- board text removed: "B18"
- board text removed: "B19"
- board text removed: "B2"
- board text removed: "B20"
- board text removed: "B21"
- board text removed: "B22"
- board text removed: "B23"
- board text removed: "B24"
- board text removed: "B25"
- board text removed: "B26"
- board text removed: "B3"
- board text removed: "B4"
- board text removed: "B5"
- board text removed: "B6"
- board text removed: "B7"
- board text removed: "B8"
- board text removed: "B9"
- board text removed: "BQ79614-1"
- board text removed: "BQ79614-2"
- board text removed: "Battery Management System V1.0"
- board text removed: "Dsigned by : Wiktor Krakowski"
- board text removed: "HV"
- board text removed: "Może nie najtaniej, ale jako tako"

Commit message: BQ1 layout complete
Parts:
- removed C47: 1uF, Capacitor_SMD:C_0603_1608Metric_Pad1.08x0.95mm_HandSolder
- moved R46 147.7 mm to (150.2, 142.7), turned to 0 degrees
- moved R33 131.3 mm to (160.9, 118.7), turned to 0 degrees
- moved R34 126.1 mm to (160.9, 122.7), turned to 0 degrees
- moved C17 122.7 mm to (172.2, 136.2), turned to 180 degrees
- moved C16 122.2 mm to (170.4, 137.7), turned to 180 degrees
- moved C18 121.1 mm to (173.9, 137.7), turned to 180 degrees
- moved R35 121.1 mm to (160.9, 126.7), turned to 0 degrees
- moved C29 120.8 mm to (165.7, 120.7)
- moved R40 118.5 mm to (150.2, 118.7), turned to 0 degrees
- moved C35 117.3 mm to (154.9, 116.7)
- moved C32 116.3 mm to (165.7, 132.7)
- moved R36 116.2 mm to (160.9, 130.7), turned to 0 degrees
- moved C30 116.1 mm to (165.7, 124.7)
- moved R41 114.0 mm to (150.2, 122.7), turned to 0 degrees
- moved C36 112.6 mm to (154.9, 120.7)
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Routing:
- net GND_HV: track 0.00 -> 66.1 mm, vias 0 -> 13
- net /Mesurements_LTC1/CB7: track 2.08 -> 66.9 mm, vias 1 -> 3
- net Net-(F13-Pad2): track 0.00 -> 63.5 mm, vias 0 -> 2
- net Net-(F14-Pad2): track 0.00 -> 62.5 mm, vias 0 -> 2
- net /Mesurements_LTC1/Battery/Batt1_+: track 0.00 -> 61.9 mm, vias 0 -> 3
- net Net-(F15-Pad2): track 0.00 -> 60.8 mm, vias 0 -> 2
- net Net-(F16-Pad2): track 0.00 -> 58.9 mm, vias 0 -> 2
- net Net-(F17-Pad2): track 0.00 -> 57.8 mm, vias 0 -> 2
- net Net-(F18-Pad2): track 0.00 -> 56.1 mm, vias 0 -> 2
- net Net-(F19-Pad2): track 0.00 -> 55.0 mm, vias 0 -> 2
- net Net-(F1-Pad2): track 0.00 -> 52.7 mm, vias 0 -> 2
- net Net-(F7-Pad2): track 0.00 -> 51.1 mm, vias 0 -> 2
- net Net-(F8-Pad2): track 0.00 -> 49.5 mm, vias 0 -> 2
- net /Mesurements_LTC1/CB0: track 2.68 -> 52.2 mm, vias 1 -> 2
- net Net-(F9-Pad2): track 0.00 -> 48.6 mm, vias 0 -> 2
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- added copper zone on F.Cu, net GND_HV
- added copper zone on In1.Cu, net GND_HV
- added copper zone on In2.Cu, net GND_HV
- added copper zone on B.Cu, net Net-(Q8-C)
- added copper zone on F.Cu, net Net-(Q8-C)
- added copper zone on In1.Cu, net Net-(Q8-C)
- added copper zone on In2.Cu, net Net-(Q8-C)
Other:
- board size 8.5 x 2 mm -> 182 x 174.8 mm
