File: Hardware/Mesurements_LTC1.kicad_sch (KiCad schematic)
At the start: 12 parts, among them Q8 100V/2W, U1 BQ79614PAPRQ1

Commit message: Bms plug and play, 2nd iteration with the same pinout
Parts:
- U1: footprint footrpint:BQ79614PAPRQ1 -> Package_QFP:Texas_TQFP-64-1EP_10x10mm_P0.5mm_EP8x8mm_Mask4.44x4.44mm_ThermalVias

Commit message: New connectors jst_xh for low voltage side of bms
Other:
- title: (none) -> Battery Management System for a high power gokart battery
Changed lines of the file:
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@@
 	(generator_version "10.0")
 	(paper "A4")
+	(title_block
+		(title "Battery Management System for a high power gokart battery")
+	)
 	(junction
 		(at 98.425 69.215)
