File: Hardware/Mesurements_LTC1.kicad_sch (KiCad schematic)
At the start: 12 parts, among them Q8 100V/2W, U1 BQ79614PAPRQ1

Commit message: No drc errors
Parts:
- added C145: 0.47uF, Capacitor_SMD:C_0603_1608Metric_Pad1.08x0.95mm_HandSolder, symbol Device:C_Small
- added D11: 60V/0.5/3A, Diode_SMD:D_SOD-123, symbol Device:D_Schottky_Small
- added F45, F46: 400mA, Fuse:Fuse_0805_2012Metric, symbol Device:Fuse_Small
- added J11: Conn_01x02, Connector_JST:JST_XH_S2B-XH-A_1x02_P2.50mm_Horizontal, symbol Connector_Generic:Conn_01x02
- added R15, R61: 300R, Resistor_SMD:R_0603_1608Metric, symbol Device:R_Small
Connections:
- net at U1.63 (BBN): now also R61.1
- net at U1.64 (BBP): now also R15.1
- new net: F46.1, J11.1 (Pin_1)
- new net: F45.1, J11.2 (Pin_2)
- new net: C145.2, D11.1 (K), F45.2, R15.2
- new net: C145.1, D11.2 (A), F46.2, R61.2
- no-connect marks 8 -> 6
