File: Hardware/Power.kicad_sch (KiCad schematic)
At the start: 2 parts, among them J18 Conn_01x02

Commit message: nearly done
Parts:
- removed TP13: TestPoint_Small, TestPoint:TestPoint_Pad_D1.0mm, symbol Connector:TestPoint_Small
Changed lines of the file:
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@@
-	)
-	(junction
-		(at 27.94 43.18)
-		(diameter 0)
-		(color 0 0 0 0)
 	)
 	(junction
@@
 	(wire
 		(pts
-			(xy 24.13 43.18) (xy 27.94 43.18)
+			(xy 24.13 43.18) (xy 49.53 43.18)
 		)
 		(stroke
@@
 		(pts
 			(xy 24.13 35.56) (xy 24.13 40.64)
-		)
-		(stroke
-			(width 0)
-			(type default)
-		)
-	)
-	(wire
-		(pts
-			(xy 27.94 43.18) (xy 49.53 43.18)
 		)
 		(stroke
@@
 			)
 		)
-	)
-	(symbol
-		(lib_id "Connector:TestPoint_Small")
-		(at 27.94 43.18 0)
-		(unit 1)
-		(body_style 1)
-		(exclude_from_sim no)
-		(in_bom yes)
-		(on_board yes)
-		(in_pos_files yes)
-		(dnp no)
-		(fields_autoplaced yes)
-		(property "Reference" "TP13"
-			(at 29.21 41.9099 0)
-			(show_name no)
-			(do_not_autoplace no)
-			(effects
-				(font
-					(size 1.27 1.27)
-				)
-				(justify left)
-			)
-		)
-		(property "Value" "TestPoint_Small"
-			(at 29.21 44.4499 0)
-			(hide yes)
-			(show_name no)
-			(do_not_autoplace no)
-			(effects
-				(font
-					(size 1.27 1.27)
-				)
-				(justify left)
-			)
-		)
-		(property "Footprint" "TestPoint:TestPoint_Pad_D1.0mm"
-			(at 33.02 43.18 0)
-			(hide yes)
-			(show_name no)
-			(do_not_autoplace no)
-			(effects
-				(font
-					(size 1.27 1.27)
-				)
-			)
-		)
-		(property "Datasheet" ""
-			(at 33.02 43.18 0)
-			(hide yes)
-			(show_name no)
-			(do_not_autoplace no)
-			(effects
-				(font
-					(size 1.27 1.27)
-				)
-			)
-		)
-		(property "Description" "test point"
-			(at 27.94 43.18 0)
-			(hide yes)
-			(show_name no)
-			(do_not_autoplace no)
-			(effects
-				(font
-					(size 1.27 1.27)
-				)
-			)
-		)
-		(pin "1"
-		)
-		(instances
-			(project "BMS"
-				(path "/26289bb6-56bc-4ca1-b1a2-18d58d1afdf5/b306fb08-ef5e-4bf5-8efa-c4e5200f566a"
-					(reference "TP13")
-					(unit 1)
-				)
-			)
-		)

Commit message: New connectors jst_xh for low voltage side of bms
Other:
- title: (none) -> Battery Management System for a high power gokart battery
Changed lines of the file:
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@@
 	(generator_version "10.0")
 	(paper "A5")
+	(title_block
+		(title "Battery Management System for a high power gokart battery")
+	)
 	(text "5V power supply\n"
 		(exclude_from_sim no)
