File: Hardware/Temperature_LTC_1.kicad_sch (KiCad schematic)
At the start: 35 parts, among them J16 Conn_01x10

Commit message: Bms plug and play, 2nd iteration with the same pinout
Parts:
- removed R15: 100k, Resistor_SMD:R_0603_1608Metric_Pad0.98x0.95mm_HandSolder, symbol Device:R_Small
- added F4, F40, F41: 400mA, Fuse:Fuse_0805_2012Metric, symbol Device:Fuse_Small
Connections:
- net GND_HV: now also F4.2, F40.2, F41.2; no longer J16.6 (Pin_6), J16.7 (Pin_7), J16.8 (Pin_8)
- new net: F40.1, J16.7 (Pin_7)
- new net: F41.1, J16.8 (Pin_8)
- new net: F4.1, J16.6 (Pin_6)

Commit message: BQ1 layout complete
Parts:
- removed C47: 1uF, Capacitor_SMD:C_0603_1608Metric_Pad1.08x0.95mm_HandSolder, symbol Device:C_Small
Changed lines of the file:
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@@
 	)
 	(junction
-		(at 123.19 30.48)
-		(diameter 0)
-		(color 0 0 0 0)
-	)
-	(junction
 		(at 189.23 100.33)
 		(diameter 0)
@@
 	(wire
 		(pts
-			(xy 123.19 30.48) (xy 133.35 30.48)
-		)
-		(stroke
-			(width 0)
-			(type default)
-		)
-	)
-	(wire
-		(pts
 			(xy 189.23 100.33) (xy 199.39 100.33)
 		)
@@
 	(wire
 		(pts
-			(xy 123.19 36.83) (xy 123.19 35.56)
-		)
-		(stroke
-			(width 0)
-			(type default)
-		)
-	)
-	(wire
-		(pts
 			(xy 184.15 40.64) (xy 189.23 40.64)
 		)
@@
 	(wire
 		(pts
-			(xy 116.84 30.48) (xy 123.19 30.48)
+			(xy 116.84 30.48) (xy 133.35 30.48)
 		)
 		(stroke
@@
 		(in_pos_files yes)
 		(dnp no)
-		(fields_autoplaced yes)
 		(property "Reference" "R10"
 			(at 120.65 153.67 90)
@@
 	)
 	(symbol
-		(lib_id "Device:C_Small")
-		(at 123.19 33.02 0)
-		(unit 1)
-		(body_style 1)
-		(exclude_from_sim no)
-		(in_bom yes)
-		(on_board yes)
-		(in_pos_files yes)
-		(dnp no)
-		(fields_autoplaced yes)
-		(property "Reference" "C47"
-			(at 125.73 31.7562 0)
-			(show_name no)
-			(do_not_autoplace no)
-			(effects
-				(font
-					(size 1.27 1.27)
-				)
-				(justify left)
-			)
-		)
-		(property "Value" "1uF"
-			(at 125.73 34.2962 0)
-			(show_name no)
-			(do_not_autoplace no)
-			(effects
-				(font
-					(size 1.27 1.27)
-				)
-				(justify left)
-			)
-		)
-		(property "Footprint" "Capacitor_SMD:C_0603_1608Metric_Pad1.08x0.95mm_HandSolder"
-			(at 123.19 33.02 0)
-			(hide yes)
-			(show_name no)
-			(do_not_autoplace no)
-			(effects
-				(font
-					(size 1.27 1.27)
-				)
-			)
-		)
-		(property "Datasheet" "https://www.mouser.pl/ProductDetail/TAIYO-YUDEN/EMK107B7105MA8T?qs=sGAEpiMZZMsh%252B1woXyUXj30ZYomYlxpXD%252BuSrqeE39U%3D"
-			(at 123.19 33.02 0)
-			(hide yes)
-			(show_name no)
-			(do_not_autoplace no)
-			(effects
-				(font
-					(size 1.27 1.27)
-				)
-			)
-		)
-		(property "Description" "Unpolarized capacitor, small symbol"
-			(at 123.19 33.02 0)
-			(hide yes)
-			(show_name no)
-			(do_not_autoplace no)
-			(effects
-				(font
-					(size 1.27 1.27)
-				)
-			)
-		)
-		(pin "1"
-		)
-		(pin "2"
-		)
-		(instances
-			(project "BMS"
-				(path "/26289bb6-56bc-4ca1-b1a2-18d58d1afdf5/329d2a9a-b359-4d8c-80ce-edb0b764c6b7/a43b6b0a-d3da-47c5-ab92-e0e154337573"
-					(reference "C47")
-					(unit 1)
-				)
-			)
-		)
-	)
-	(symbol
 		(lib_id "power:GND")
 		(at 115.57 168.91 0)
@@
 					(unit 1)
 				)
-			)
-		)
-	)
-	(symbol
-		(lib_id "power:GND")
-		(at 123.19 36.83 270)
-		(unit 1)
-		(body_style 1)
-		(exclude_from_sim no)
-		(in_bom yes)
-		(on_board yes)
-		(in_pos_files yes)
-		(dnp no)
-		(property "Reference" "#PWR042"
-			(at 116.84 36.83 0)
-			(hide yes)
-			(show_name no)
-			(do_not_autoplace no)
-			(effects
-				(font
-					(size 1.27 1.27)
-				)
-			)
-		)
-		(property "Value" "GND_HV"
-			(at 119.38 36.83 90)
-			(show_name no)
-			(do_not_autoplace no)
-			(effects
-				(font
-					(size 1.27 1.27)
-				)
-				(justify right)
-			)
-		)
-		(property "Footprint" ""
-			(at 123.19 36.83 0)
-			(hide yes)
-			(show_name no)
-			(do_not_autoplace no)
-			(effects
-				(font
-					(size 1.27 1.27)
-				)
-			)
-		)
-		(property "Datasheet" ""
-			(at 123.19 36.83 0)
-			(hide yes)
-			(show_name no)
-			(do_not_autoplace no)
-			(effects
-				(font
-					(size 1.27 1.27)
-				)
-			)
-		)
-		(property "Description" "Power symbol creates a global label with name \"GND\" , ground"
-			(at 123.19 36.83 0)
-			(hide yes)
-			(show_name no)
-			(do_not_autoplace no)
-			(effects
-				(font
-					(size 1.27 1.27)
-				)
-			)
-		)
-		(pin "1"
-		)
-		(instances
-			(project "BMS"
-				(path "/26289bb6-56bc-4ca1-b1a2-18d58d1afdf5/329d2a9a-b359-4d8c-80ce-edb0b764c6b7/a43b6b0a-d3da-47c5-ab92-e0e154337573"
-					(reference "#PWR042")
-					(unit 1)
-				)

Commit message: New connectors jst_xh for low voltage side of bms
Other:
- title: (none) -> Battery Management System for a high power gokart battery
Changed lines of the file:
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@@
 	(generator_version "10.0")
 	(paper "A4")
+	(title_block
+		(title "Battery Management System for a high power gokart battery")
+	)
 	(junction
 		(at 129.54 100.33)

Commit message: No drc errors
Parts:
- removed F4, F40, F41: 400mA, Fuse:Fuse_0805_2012Metric, symbol Device:Fuse_Small
- removed J16: Conn_01x10, footrpint:HARWIN_G125-MV11005L1P, symbol Connector_Generic:Conn_01x10
- removed TH1: 10k b= 3000, Resistor_SMD:R_0603_1608Metric_Pad0.98x0.95mm_HandSolder, symbol Device:Thermistor_NTC
- added J19: B16B-PUDSS-1(LF)(SN), Connector_JST:JST_PUD_B16B-PUDSS_2x08_P2.00mm_Vertical, symbol Connector_Generic:Conn_02x08_Odd_Even
- added TH17: 10k b= 3000, symbol Device:Thermistor_NTC
Connections:
- net GND_HV: now also J19.1 (Pin_1), J19.11 (Pin_11), J19.13 (Pin_13), J19.15 (Pin_15), J19.3 (Pin_3), J19.5 (Pin_5), J19.7 (Pin_7), J19.9 (Pin_9), TH17.2
- net Thermistor2: now also J19.4 (Pin_4)
- net Thermistor3: now also J19.6 (Pin_6)
- net Thermistor4: now also J19.8 (Pin_8)
- net Thermistor5: now also J19.10 (Pin_10)
- net Thermistor6: now also J19.12 (Pin_12)
- net Thermistor7: now also J19.14 (Pin_14)
- net Thermistor8: now also J19.16 (Pin_16)
- net Thermistor1: now reaches R14.2, R8.2
- net Thermistor1: now also J19.2 (Pin_2), TH17.1
