File: Hardware/Temperature_LTC_2.kicad_sch (KiCad schematic)
At the start: 35 parts, among them J10 Conn_01x10

Commit message: Bms plug and play, 2nd iteration with the same pinout
Parts:
- removed R101: 100k, Resistor_SMD:R_0603_1608Metric_Pad0.98x0.95mm_HandSolder, symbol Device:R_Small
- added F42, F43, F44: 400mA, Fuse:Fuse_0805_2012Metric, symbol Device:Fuse_Small
Connections:
- net GND_HV2: now also F42.2, F43.2, F44.2; no longer J10.6 (Pin_6), J10.7 (Pin_7), J10.8 (Pin_8)
- new net: F42.1, J10.6 (Pin_6)
- new net: F43.1, J10.7 (Pin_7)
- new net: F44.1, J10.8 (Pin_8)

Commit message: nearly done
Parts:
- removed C71: 1uF, Capacitor_SMD:C_0603_1608Metric_Pad1.08x0.95mm_HandSolder, symbol Device:C_Small
Changed lines of the file:
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@@
 	)
 	(junction
-		(at 115.57 20.32)
-		(diameter 0)
-		(color 0 0 0 0)
-	)
-	(junction
 		(at 120.65 115.57)
 		(diameter 0)
@@
 	(wire
 		(pts
-			(xy 115.57 20.32) (xy 125.73 20.32)
+			(xy 109.22 20.32) (xy 125.73 20.32)
 		)
 		(stroke
@@
 	(wire
 		(pts
-			(xy 109.22 20.32) (xy 115.57 20.32)
-		)
-		(stroke
-			(width 0)
-			(type default)
-		)
-	)
-	(wire
-		(pts
 			(xy 116.84 90.17) (xy 121.92 90.17)
 		)
@@
 	(wire
 		(pts
-			(xy 115.57 26.67) (xy 115.57 25.4)
-		)
-		(stroke
-			(width 0)
-			(type default)
-		)
-	)
-	(wire
-		(pts
 			(xy 120.65 148.59) (xy 130.81 148.59)
 		)
@@
 	)
 	(symbol
-		(lib_id "Device:C_Small")
-		(at 115.57 22.86 0)
-		(unit 1)
-		(body_style 1)
-		(exclude_from_sim no)
-		(in_bom yes)
-		(on_board yes)
-		(in_pos_files yes)
-		(dnp no)
-		(fields_autoplaced yes)
-		(property "Reference" "C71"
-			(at 118.11 21.5962 0)
-			(show_name no)
-			(do_not_autoplace no)
-			(effects
-				(font
-					(size 1.27 1.27)
-				)
-				(justify left)
-			)
-		)
-		(property "Value" "1uF"
-			(at 118.11 24.1362 0)
-			(show_name no)
-			(do_not_autoplace no)
-			(effects
-				(font
-					(size 1.27 1.27)
-				)
-				(justify left)
-			)
-		)
-		(property "Footprint" "Capacitor_SMD:C_0603_1608Metric_Pad1.08x0.95mm_HandSolder"
-			(at 115.57 22.86 0)
-			(hide yes)
-			(show_name no)
-			(do_not_autoplace no)
-			(effects
-				(font
-					(size 1.27 1.27)
-				)
-			)
-		)
-		(property "Datasheet" "https://www.mouser.pl/ProductDetail/TAIYO-YUDEN/EMK107B7105MA8T?qs=sGAEpiMZZMsh%252B1woXyUXj30ZYomYlxpXD%252BuSrqeE39U%3D"
-			(at 115.57 22.86 0)
-			(hide yes)
-			(show_name no)
-			(do_not_autoplace no)
-			(effects
-				(font
-					(size 1.27 1.27)
-				)
-			)
-		)
-		(property "Description" "Unpolarized capacitor, small symbol"
-			(at 115.57 22.86 0)
-			(hide yes)
-			(show_name no)
-			(do_not_autoplace no)
-			(effects
-				(font
-					(size 1.27 1.27)
-				)
-			)
-		)
-		(pin "1"
-		)
-		(pin "2"
-		)
-		(instances
-			(project "BMS"
-				(path "/26289bb6-56bc-4ca1-b1a2-18d58d1afdf5/99f7ea83-6836-44ea-889b-f0d453e84b38/ebf36db7-cdb4-471e-a54c-71c0b45a68a4"
-					(reference "C71")
-					(unit 1)
-				)
-			)
-		)
-	)
-	(symbol
 		(lib_id "Device:Fuse_Small")
 		(at 50.165 76.2 0)
@@
 					(unit 1)
 				)
-			)
-		)
-	)
-	(symbol
-		(lib_id "power:GND")
-		(at 115.57 26.67 270)
-		(unit 1)
-		(body_style 1)
-		(exclude_from_sim no)
-		(in_bom yes)
-		(on_board yes)
-		(in_pos_files yes)
-		(dnp no)
-		(property "Reference" "#PWR066"
-			(at 109.22 26.67 0)
-			(hide yes)
-			(show_name no)
-			(do_not_autoplace no)
-			(effects
-				(font
-					(size 1.27 1.27)
-				)
-			)
-		)
-		(property "Value" "GND_HV2"
-			(at 111.76 26.67 90)
-			(show_name no)
-			(do_not_autoplace no)
-			(effects
-				(font
-					(size 1.27 1.27)
-				)
-				(justify right)
-			)
-		)
-		(property "Footprint" ""
-			(at 115.57 26.67 0)
-			(hide yes)
-			(show_name no)
-			(do_not_autoplace no)
-			(effects
-				(font
-					(size 1.27 1.27)
-				)
-			)
-		)
-		(property "Datasheet" ""
-			(at 115.57 26.67 0)
-			(hide yes)
-			(show_name no)
-			(do_not_autoplace no)
-			(effects
-				(font
-					(size 1.27 1.27)
-				)
-			)
-		)
-		(property "Description" "Power symbol creates a global label with name \"GND\" , ground"
-			(at 115.57 26.67 0)
-			(hide yes)
-			(show_name no)
-			(do_not_autoplace no)
-			(effects
-				(font
-					(size 1.27 1.27)
-				)
-			)
-		)
-		(pin "1"
-		)
-		(instances
-			(project "BMS"
-				(path "/26289bb6-56bc-4ca1-b1a2-18d58d1afdf5/99f7ea83-6836-44ea-889b-f0d453e84b38/ebf36db7-cdb4-471e-a54c-71c0b45a68a4"
-					(reference "#PWR066")
-					(unit 1)
-				)

Commit message: New connectors jst_xh for low voltage side of bms
Other:
- title: (none) -> Battery Management System for a high power gokart battery
Changed lines of the file:
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@@
 	(generator_version "10.0")
 	(paper "A4")
+	(title_block
+		(title "Battery Management System for a high power gokart battery")
+	)
 	(junction
 		(at 181.61 90.17)

Commit message: No drc errors
Parts:
- removed F42, F43, F44: 400mA, Fuse:Fuse_0805_2012Metric, symbol Device:Fuse_Small
- removed J10: Conn_01x10, footrpint:HARWIN_G125-MV11005L1P, symbol Connector_Generic:Conn_01x10
- added J25: B16B-PUDSS-1(LF)(SN), Connector_JST:JST_PUD_B16B-PUDSS_2x08_P2.00mm_Vertical, symbol Connector_Generic:Conn_02x08_Odd_Even
- TH13: now not fitted; now left out of the parts list
Connections:
- net GND_HV2: now also J25.1 (Pin_1), J25.11 (Pin_11), J25.13 (Pin_13), J25.15 (Pin_15), J25.3 (Pin_3), J25.5 (Pin_5), J25.7 (Pin_7), J25.9 (Pin_9)
- net Thermistor1: now also J25.2 (Pin_2)
- net Thermistor2: now also J25.4 (Pin_4)
- net Thermistor3: now also J25.6 (Pin_6)
- net Thermistor4: now also J25.8 (Pin_8)
- net Thermistor5: now also J25.10 (Pin_10)
- net Thermistor6: now also J25.12 (Pin_12)
- net Thermistor7: now also J25.14 (Pin_14)
- net Thermistor8: now also J25.16 (Pin_16)
