File: Hardware/Power_3.3V.kicad_sch (KiCad schematic)
At the start: 14 parts, among them IC3 TPS563200DDCR

Commit message: Wysłane do JLC
Parts:
- L2: footprint Inductor_SMD:L_Sunlord_MWSA0402S -> Inductor_SMD:L_TDK_VLS6045EX_VLS6045AF
