File: BMS Master/STM.kicad_sch (KiCad schematic)
At the start: 12 parts, among them IC1 STM32H742VIT6

Commit message: Prace nad masterem
Parts:
- removed C1: 100n ceramiczny, Capacitor_SMD:C_0603_1608Metric_Pad1.08x0.95mm_HandSolder, symbol Device:C_Small
- removed C141: 47n, Capacitor_SMD:C_0603_1608Metric_Pad1.08x0.95mm_HandSolder, symbol Device:C_Small
- removed C66, C67, C68, C69, C70: 1uF, Capacitor_SMD:C_0603_1608Metric_Pad1.08x0.95mm_HandSolder, symbol Device:C_Small
- added C11, C12, C13, C14, C15, C16, C17: CC0603KRX7R9BB104, Capacitor_SMD:C_0603_1608Metric, symbol Device:C_Small
- added D10, D11, D12, D9: KT-0603R, LED_SMD:LED_0603_1608Metric, symbol Device:LED_Small
- added R20, R21, R22, R23: 0603WAF1000T5E, Resistor_SMD:R_0603_1608Metric, symbol Device:R_Small
Connections:
- net GND: now also C11.2, C12.1, C13.1, C14.2, C15.2, C16.2, C17.2
- net Input4: now reaches IC1.43 (PE13)
- net +3.3V renamed +3V3
- net +3V3: now also C12.2, C13.2, C14.1, C15.1, C16.1, R20.1, R21.1, R22.1, R23.1; no longer IC1.6 (VBAT), IC1.75 (VDD_4)
- net Button2 renamed Input1
- net Button3 renamed Input2
- net Button4 renamed Input3
- net Curr_sense: no longer names the net of IC1.32 (PC4)
- net Curr_sense2: no longer names the net of IC1.35 (PB1)
- net ERROR: no longer names the net of IC1.1 (PE2)
- net ERROR: now also D9.1 (K)
- net LED1: no longer names the net of IC1.2 (PE3)
- net LED1: now also D10.1 (K)
- net LED2: no longer names the net of IC1.3 (PE4)
- net LED2: now also D11.1 (K)
- net LED3: no longer names the net of IC1.4 (PE5)
- net LED3: now also D12.1 (K)
- net RX_1 renamed RX MISO
- net TX_1 renamed TX MOSI
- new net: D10.2 (A), R21.2
- new net: D12.2 (A), R23.2
- new net: D11.2 (A), R22.2
- new net: D9.2 (A), R20.2
- new net 3.3V_IN: C11.1, C17.1, IC1.6 (VBAT), IC1.75 (VDD_4)
- no-connect marks 60 -> 59
Other:
- note removed: "Curr_sense is connected to ADC"
- note removed: "tego nie pewny"
