File: BMS_Slave/BMS_Slave.kicad_pcb (KiCad board)
At the start: 4 copper layers, 93.2 x 92.8 mm, 155 parts, among them J1 Conn_01x01_Socket, J10 Batt 7, J11 Batt 6, J12 Batt 2, J13 Batt 5, J14 Batt 1, J15 Batt 0, J16 Conn_01x01_Socket, J17 Conn_01x01_Socket, J18 Conn_01x01_Socket, J19 Conn_01x01_Socket, J2 Batt 13, J20 Conn_01x01_Socket, J21 Conn_01x01_Socket, J22 Conn_01x01_Socket, J23 Conn_01x01_Socket, J24 Conn_01x01_Socket, J25 Conn_01x01_Socket, J26 Conn_01x01_Socket, J27 Conn_01x01_Socket, J28 Conn_01x01_Socket, J29 Conn_01x01_Socket, J3 Batt 12, J30 Conn_01x01_Socket, J33 Dsub 9, J34 Dsub 9, J4 Batt 11, J5 Batt 10, J6 Batt 9, J7 Batt 8, J8 Batt 4, J9 Batt 3, Q8 FZT653TA, T2 TM0608SR, T3 TM0608SR, U1 BQ79614PAPRQ1

Commit message: Dodano connectory hińskie zamiast padów, kontynuacja layoutu
Parts:
- removed J1, J16, J17, J18, J19, J20, J21, J22, J23, J24, J25, J26, J27, J28, J29, J30: Conn_01x01_Socket, Connector_Wire:SolderWirePad_1x01_SMD_2x4mm
- removed J14: Batt 1, Connector_Wire:SolderWirePad_1x01_SMD_5x10mm
- removed J15: Batt 0, Connector_Wire:SolderWirePad_1x01_SMD_5x10mm
- removed J33, J34: Dsub 9, Connector_Dsub:DSUB-9_Pins_Vertical_P2.77x2.84mm_MountingHoles
- added F19: 0.5A resetable, Fuse:Fuse_0805_2012Metric, F.Cu at (169.6, 55.1)
- added F20: 0.5A resetable, Fuse:Fuse_0805_2012Metric, F.Cu at (169.6, 58.1)
- added F21: 0.5A resetable, Fuse:Fuse_0805_2012Metric, F.Cu at (164.0, 70.9)
- added F22: 0.5A resetable, Fuse:Fuse_0805_2012Metric, F.Cu at (146.7, 43.5)
- added F23: 0.5A resetable, Fuse:Fuse_0805_2012Metric, F.Cu at (158.2, 30.8)
- added F24: 0.5A resetable, Fuse:Fuse_0805_2012Metric, F.Cu at (169.6, 30.8)
- added F25: 0.5A resetable, Fuse:Fuse_0805_2012Metric, F.Cu at (146.7, 56.3)
- added F26: 0.5A resetable, Fuse:Fuse_0805_2012Metric, F.Cu at (169.6, 43.5)
- added F27: 0.5A resetable, Fuse:Fuse_0805_2012Metric, F.Cu at (158.2, 56.3)
- added F28: 0.5A resetable, Fuse:Fuse_0805_2012Metric, F.Cu at (158.2, 43.5)
- added R3: 300, Resistor_SMD:R_0603_1608Metric, F.Cu at (140.5, 81.5)
- added R6: 300, Resistor_SMD:R_0603_1608Metric, F.Cu at (142.0, 81.5)
- J10: value Batt 7 -> SH-XH2.54-2P; footprint Connector_Wire:SolderWirePad_1x01_SMD_5x10mm -> Connector_JST:JST_XH_B2B-XH-A_1x02_P2.50mm_Vertical
- J11: value Batt 6 -> SH-XH2.54-2P; footprint Connector_Wire:SolderWirePad_1x01_SMD_5x10mm -> Connector_JST:JST_XH_B2B-XH-A_1x02_P2.50mm_Vertical
- J12: value Batt 2 -> SH-XH2.54-2P; footprint Connector_Wire:SolderWirePad_1x01_SMD_5x10mm -> Connector_JST:JST_XH_B2B-XH-A_1x02_P2.50mm_Vertical
- J13: value Batt 5 -> B2B-PH-K-S-GW; footprint Connector_Wire:SolderWirePad_1x01_SMD_5x10mm -> Model:CONN2_B2B-PH-K-S_JST
- J2: value Batt 13 -> Conn_01x14; footprint Connector_Wire:SolderWirePad_1x01_SMD_5x10mm -> Conn_custom:XY-XHB2.54-14A21
- J3: value Batt 12 -> B2B-PH-K-S-GW; footprint Connector_Wire:SolderWirePad_1x01_SMD_5x10mm -> Model:CONN2_B2B-PH-K-S_JST
- J4: value Batt 11 -> B2B-PH-K-S-GW; footprint Connector_Wire:SolderWirePad_1x01_SMD_5x10mm -> Model:CONN2_B2B-PH-K-S_JST
- J5: value Batt 10 -> SH-XH2.54-2P; footprint Connector_Wire:SolderWirePad_1x01_SMD_5x10mm -> Connector_JST:JST_XH_B2B-XH-A_1x02_P2.50mm_Vertical
- J6: value Batt 9 -> SH-XH2.54-2P; footprint Connector_Wire:SolderWirePad_1x01_SMD_5x10mm -> Connector_JST:JST_XH_B2B-XH-A_1x02_P2.50mm_Vertical
- J7: value Batt 8 -> SH-XH2.54-2P; footprint Connector_Wire:SolderWirePad_1x01_SMD_5x10mm -> Connector_JST:JST_XH_B2B-XH-A_1x02_P2.50mm_Vertical
- J8: value Batt 4 -> SH-XH2.54-2P; footprint Connector_Wire:SolderWirePad_1x01_SMD_5x10mm -> Connector_JST:JST_XH_B2B-XH-A_1x02_P2.50mm_Vertical
- J9: value Batt 3 -> SH-XH2.54-2P; footprint Connector_Wire:SolderWirePad_1x01_SMD_5x10mm -> Connector_JST:JST_XH_B2B-XH-A_1x02_P2.50mm_Vertical
- moved F18 131.0 mm to (78.5, 107.8), turned to 180 degrees
- moved F9 118.8 mm to (78.5, 69.8), turned to 180 degrees
- moved F7 102.1 mm to (78.4, 94.5)
- moved F10 99.8 mm to (78.5, 89.5)
- moved J2 98.6 mm to (72.4, 88.2), turned to -90 degrees
- moved J4 91.9 mm to (107.8, 110.0), turned to 90 degrees
- moved R39 91.4 mm to (91.8, 94.5)
- moved R41 88.5 mm to (91.8, 89.5)
- moved F13 88.1 mm to (78.5, 82.0)
- moved F6 87.7 mm to (78.5, 97.0)
- moved F8 85.0 mm to (78.5, 91.8)
- moved F14 74.9 mm to (78.5, 79.5)
- moved F16 73.3 mm to (78.5, 74.5)
- moved F3 70.9 mm to (78.5, 105.0)
- moved R38 67.6 mm to (101.8, 97.2)
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Connections:
- net /Temperature_LTC_1/T1 renamed /Temperature/T1
- net /Temperature_LTC_1/T2 renamed /Temperature/T2
- net /Temperature_LTC_1/T3 renamed /Temperature/T3
- net /Temperature_LTC_1/T4 renamed /Temperature/T4
- net /Temperature_LTC_1/T5 renamed /Temperature/T5
- net /Temperature_LTC_1/T6 renamed /Temperature/T6
- net /Temperature_LTC_1/T7 renamed /Temperature/T7
- net /Temperature_LTC_1/T8 renamed /Temperature/T8
- net /Temperature_LTC_1/TSREF renamed /Temperature/TSREF
- C24 pad 1: /Battery/Array3/VC_LOWER -> /VC1
- C25 pad 1: /Battery/Array3/CB_LOWER -> /CB1
- C36 pad 1: /Battery/Array9/VC_LOWER -> /VC7
- C37 pad 1: /Battery/Array9/CB_LOWER -> /CB7
- C48 pad 1: /IIC- -> /dp4-
- C49 pad 1: /IIC+ -> /dp4+
- C51 pad 1: /IIC+ -> /dp3+
- C52 pad 1: /IIC- -> /dp3-
- J10 pad 1: /Battery/Array8/CELL -> Net-(J10-Pin_1)
- J11 pad 1: /Battery/Array7/CELL -> Net-(J11-Pin_1)
- J12 pad 1: /Battery/Array3/CELL -> Net-(J12-Pin_1)
- J13 pad 1: /Battery/Array6/CELL -> Net-(J13-Pin_1)
- J2 pad 1: /Battery/Array14/CELL -> /Battery/Array1/CELL
- J3 pad 1: /Battery/Array13/CELL -> /dp1+
- J4 pad 1: /Battery/Array12/CELL -> /dp6+
- J5 pad 1: /Battery/Array11/CELL -> Net-(J5-Pin_1)
- J6 pad 1: /Battery/Array10/CELL -> Net-(J6-Pin_1)
- J7 pad 1: /Battery/Array9/CELL -> Net-(J7-Pin_1)
- J8 pad 1: /Battery/Array5/CELL -> Net-(J8-Pin_1)
- J9 pad 1: /Battery/Array4/CELL -> Net-(J9-Pin_1)
- R58 pad 1: /IIC- -> /dp4-
- R58 pad 2: /IIC+ -> /dp4+
- R59 pad 2: Net-(J1-Pin_1) -> Net-(J5-Pin_1)
- R60 pad 1: Net-(J1-Pin_1) -> Net-(J5-Pin_1)
- R61 pad 2: Net-(J17-Pin_1) -> Net-(J6-Pin_1)
- R62 pad 1: Net-(J17-Pin_1) -> Net-(J6-Pin_1)
- R63 pad 2: Net-(J19-Pin_1) -> Net-(J7-Pin_1)
- R64 pad 1: Net-(J19-Pin_1) -> Net-(J7-Pin_1)
- R65 pad 2: Net-(J21-Pin_1) -> Net-(J8-Pin_1)
- R66 pad 1: Net-(J21-Pin_1) -> Net-(J8-Pin_1)
- R67 pad 2: Net-(J23-Pin_1) -> Net-(J9-Pin_1)
- R68 pad 1: Net-(J23-Pin_1) -> Net-(J9-Pin_1)
- R69 pad 2: Net-(J25-Pin_1) -> Net-(J10-Pin_1)
- R70 pad 1: Net-(J25-Pin_1) -> Net-(J10-Pin_1)
- R71 pad 2: Net-(J27-Pin_1) -> Net-(J11-Pin_1)
- R72 pad 1: Net-(J27-Pin_1) -> Net-(J11-Pin_1)
- R73 pad 2: Net-(J29-Pin_1) -> Net-(J12-Pin_1)
- R74 pad 1: Net-(J29-Pin_1) -> Net-(J12-Pin_1)
- R75 pad 1: /IIC+ -> /dp4+
- R75 pad 2: /ILC+ -> /dp5+
- R76 pad 1: /ILC- -> /dp5-
- R76 pad 2: /IIC- -> /dp4-
- R77 pad 1: /IIC- -> /dp3-
- R77 pad 2: /IIC+ -> /dp3+
- R78 pad 1: /IIC+ -> /dp3+
- R78 pad 2: /ILC+ -> /dp2+
- R79 pad 1: /ILC- -> /dp2-
- R79 pad 2: /IIC- -> /dp3-
- T2 pad 1: Net-(J33-Pin_7) -> /dp1-
- T2 pad 3: Net-(J33-Pin_2) -> /dp1+
- T2 pad 4: /ILC- -> /dp2+
- T2 pad 6: /ILC+ -> /dp2-
- T3 pad 1: Net-(J34-Pin_7) -> /dp6+
- T3 pad 3: Net-(J34-Pin_2) -> /dp6-
- T3 pad 4: /ILC- -> /dp5-
- T3 pad 6: /ILC+ -> /dp5+
- U1 pad 36: GND_HV -> GND
- U1 pad 40: /IIC+ -> /dp4+
- U1 pad 41: /IIC- -> /dp4-
- U1 pad 42: /IIC- -> /dp3-
- U1 pad 43: /IIC+ -> /dp3+
- U1 pad 46: GND_HV -> GND
- U1 pad 50: GND_HV -> GND
- U1 pad 63: unconnected-(U1-BBN-Pad63) -> Net-(U1-BBN)
- U1 pad 64: unconnected-(U1-BBP-Pad64) -> Net-(U1-BBP)
Routing:
- net GND: track 0.00 -> 150.1 mm, vias 0 -> 113
- net Net-(F17-Pad2): track 0.00 -> 67.4 mm, vias 0 -> 2
- net /CB12: track 0.00 -> 66.5 mm
- net Net-(F16-Pad2): track 0.00 -> 65.0 mm, vias 0 -> 2
- net Net-(F15-Pad2): track 0.00 -> 60.4 mm, vias 0 -> 2
- net /CB10: track 0.00 -> 59.8 mm
- net Net-(F14-Pad2): track 0.00 -> 59.0 mm, vias 0 -> 2
- net /CB13: track 0.00 -> 58.2 mm
- net Net-(F13-Pad2): track 0.00 -> 56.1 mm, vias 0 -> 2
- net Net-(F12-Pad2): track 0.00 -> 53.6 mm, vias 0 -> 2
- net /CB11: track 0.00 -> 51.8 mm
- net /CB8: track 0.00 -> 51.4 mm
- net /Temperature/TSREF: track 0.00 -> 48.4 mm, vias 0 -> 9
- net /CB9: track 0.00 -> 46.2 mm
- net /CB6: track 0.00 -> 43.5 mm
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- added copper zone on F.Cu, net Net-(Q8-C)
- added copper zone on In1.Cu, net Net-(Q8-C)
- added copper zone on In2.Cu, net Net-(Q8-C)
- removed copper zone on B.Cu, net GND
- removed copper zone on F.Cu, net GND
Other:
- board size 93.2 x 92.8 mm -> 240 x 50 mm

Commit message: Zostały małe poprawki na silkscreenie i otwory montażowe
Parts:
- removed F25, F26, F27, F28: 0.5A resetable, Fuse:Fuse_0805_2012Metric
- removed J10, J11, J12, J6, J7, J8, J9: SH-XH2.54-2P, Connector_JST:JST_XH_B2B-XH-A_1x02_P2.50mm_Vertical
- added D1: Red, LED_SMD:LED_0603_1608Metric, F.Cu at (145.0, 71.8)
- added R1: 1k, Resistor_SMD:R_0603_1608Metric, F.Cu at (142.8, 71.0)
- J5: value SH-XH2.54-2P -> C66560; footprint Connector_JST:JST_XH_B2B-XH-A_1x02_P2.50mm_Vertical -> Connector_JST:JST_PHD_B16B-PHDSS_2x08_P2.00mm_Vertical
- moved F23 57.4 mm to (162.0, 88.0), turned to 90 degrees
- moved F24 53.8 mm to (162.0, 84.0), turned to 90 degrees
- moved F22 50.9 mm to (162.0, 92.0), turned to 90 degrees
- moved J13 29.3 mm to (158.5, 76.0), turned to 90 degrees
- moved J5 25.6 mm to (156.8, 97.0), turned to 90 degrees
- moved F21 25.2 mm to (162.0, 96.0), turned to 90 degrees
- moved F19 18.9 mm to (160.5, 71.8), turned to 90 degrees
- moved F20 17.7 mm to (158.5, 71.8), turned to 90 degrees
- moved R40 0.33 mm to (102.0, 92.0)
Connections:
- F21 pad 1: Net-(J5-Pin_2) -> Net-(J5-Pin_10)
- F22 pad 1: Net-(J6-Pin_2) -> Net-(J5-Pin_11)
- F23 pad 1: Net-(J7-Pin_2) -> Net-(J5-Pin_13)
- F24 pad 1: Net-(J8-Pin_2) -> Net-(J5-Pin_15)
- J5 pad 1: Net-(J5-Pin_1) -> /Temperature/Thermistor7/Thermistor
- J5 pad 2: Net-(J5-Pin_2) -> /Temperature/Thermistor6/Thermistor
- R2 pad 1: /Batt1_+ -> /Battery/Batt+
- R4 pad 1: /Batt1_+ -> /Battery/Batt+
- R59 pad 2: Net-(J5-Pin_1) -> /Temperature/Thermistor/Thermistor
- R60 pad 1: Net-(J5-Pin_1) -> /Temperature/Thermistor/Thermistor
- R61 pad 2: Net-(J6-Pin_1) -> /Temperature/Thermistor1/Thermistor
- R62 pad 1: Net-(J6-Pin_1) -> /Temperature/Thermistor1/Thermistor
- R63 pad 2: Net-(J7-Pin_1) -> /Temperature/Thermistor2/Thermistor
- R64 pad 1: Net-(J7-Pin_1) -> /Temperature/Thermistor2/Thermistor
- R65 pad 2: Net-(J8-Pin_1) -> /Temperature/Thermistor3/Thermistor
- R66 pad 1: Net-(J8-Pin_1) -> /Temperature/Thermistor3/Thermistor
- R67 pad 2: Net-(J9-Pin_1) -> /Temperature/Thermistor4/Thermistor
- R68 pad 1: Net-(J9-Pin_1) -> /Temperature/Thermistor4/Thermistor
- R69 pad 2: Net-(J10-Pin_1) -> /Temperature/Thermistor5/Thermistor
- R70 pad 1: Net-(J10-Pin_1) -> /Temperature/Thermistor5/Thermistor
- R71 pad 2: Net-(J11-Pin_1) -> /Temperature/Thermistor6/Thermistor
- R72 pad 1: Net-(J11-Pin_1) -> /Temperature/Thermistor6/Thermistor
- R73 pad 2: Net-(J12-Pin_1) -> /Temperature/Thermistor7/Thermistor
- R74 pad 1: Net-(J12-Pin_1) -> /Temperature/Thermistor7/Thermistor
Routing:
- net GND: track 150.1 -> 251.0 mm, vias 113 -> 176
- net /Battery/Batt+: track 0.00 -> 94.4 mm, vias 0 -> 3
- net Net-(F19-Pad2): track 0.00 -> 31.6 mm, vias 0 -> 2
- net Net-(F20-Pad2): track 0.00 -> 27.2 mm, vias 0 -> 2
- net /Batt1_+: track 18.8 -> 0.00 mm, vias 2 -> 0
- net /Temperature/Thermistor/Thermistor: track 0.00 -> 17.3 mm
- net /Temperature/Thermistor1/Thermistor: track 0.00 -> 16.8 mm
- net /Temperature/Thermistor2/Thermistor: track 0.00 -> 15.4 mm
- net /Temperature/Thermistor4/Thermistor: track 0.00 -> 14.5 mm
- net /Temperature/Thermistor3/Thermistor: track 0.00 -> 14.3 mm
- net /Temperature/Thermistor5/Thermistor: track 0.00 -> 12.4 mm
- net /Temperature/Thermistor6/Thermistor: track 0.00 -> 11.2 mm
- net /Temperature/TSREF: track 48.4 -> 59.6 mm
- net /Temperature/Thermistor7/Thermistor: track 0.00 -> 10.5 mm
- net Net-(J5-Pin_1): track 10.1 -> 0.00 mm
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- added copper zone on F.Cu, net /CB0
- added copper zone on In1.Cu, net /CB0
- added copper zone on In2.Cu, net /CB0
- added copper zone on F.Cu, net /CB1
- added copper zone on In1.Cu, net /CB1
- added copper zone on In2.Cu, net /CB1
- added copper zone on F.Cu, net /CB10
- added copper zone on In1.Cu, net /CB10
- added copper zone on In2.Cu, net /CB10
- added copper zone on F.Cu, net /CB11
- added copper zone on In1.Cu, net /CB11
- added copper zone on In2.Cu, net /CB11
- added copper zone on F.Cu, net /CB12
- added copper zone on In1.Cu, net /CB12
- added copper zone on In2.Cu, net /CB12
- added copper zone on F.Cu, net /CB13
- added copper zone on In1.Cu, net /CB13
- added copper zone on In2.Cu, net /CB13
- added copper zone on F.Cu, net /CB2
- added copper zone on In1.Cu, net /CB2
- added copper zone on In2.Cu, net /CB2
- added copper zone on F.Cu, net /CB3
- added copper zone on In1.Cu, net /CB3
- added copper zone on In2.Cu, net /CB3
- added copper zone on F.Cu, net /CB4
- added copper zone on In1.Cu, net /CB4
- added copper zone on In2.Cu, net /CB4
- added copper zone on F.Cu, net /CB5
- added copper zone on In1.Cu, net /CB5
- added copper zone on In2.Cu, net /CB5
- added copper zone on F.Cu, net /CB6
- added copper zone on In1.Cu, net /CB6
- added copper zone on In2.Cu, net /CB6
- added copper zone on F.Cu, net /CB7
- added copper zone on In1.Cu, net /CB7
- added copper zone on In2.Cu, net /CB7
- added copper zone on F.Cu, net /CB8
- added copper zone on In1.Cu, net /CB8
- added copper zone on In2.Cu, net /CB8
- added copper zone on F.Cu, net /CB9
- added copper zone on In1.Cu, net /CB9
- added copper zone on In2.Cu, net /CB9
- added copper zone on F.Cu, net Net-(F10-Pad2)
- added copper zone on In1.Cu, net Net-(F10-Pad2)
- added copper zone on In2.Cu, net Net-(F10-Pad2)
- added copper zone on F.Cu, net Net-(F11-Pad2)
- added copper zone on In1.Cu, net Net-(F11-Pad2)
- added copper zone on In2.Cu, net Net-(F11-Pad2)
- added copper zone on F.Cu, net Net-(F12-Pad2)
- added copper zone on In1.Cu, net Net-(F12-Pad2)
- added copper zone on In2.Cu, net Net-(F12-Pad2)
- added copper zone on F.Cu, net Net-(F13-Pad2)
- added copper zone on In1.Cu, net Net-(F13-Pad2)
- added copper zone on In2.Cu, net Net-(F13-Pad2)
- added copper zone on F.Cu, net Net-(F14-Pad2)
- added copper zone on In1.Cu, net Net-(F14-Pad2)
- added copper zone on In2.Cu, net Net-(F14-Pad2)
- added copper zone on F.Cu, net Net-(F15-Pad2)
- added copper zone on In1.Cu, net Net-(F15-Pad2)
- added copper zone on In2.Cu, net Net-(F15-Pad2)
- added copper zone on F.Cu, net Net-(F16-Pad2)
- added copper zone on In1.Cu, net Net-(F16-Pad2)
- added copper zone on In2.Cu, net Net-(F16-Pad2)
- added copper zone on F.Cu, net Net-(F17-Pad2)
- added copper zone on In1.Cu, net Net-(F17-Pad2)
- added copper zone on In2.Cu, net Net-(F17-Pad2)
- added copper zone on F.Cu, net Net-(F3-Pad2)
- added copper zone on In1.Cu, net Net-(F3-Pad2)
- added copper zone on In2.Cu, net Net-(F3-Pad2)
- added copper zone on F.Cu, net Net-(F4-Pad2)
- added copper zone on In1.Cu, net Net-(F4-Pad2)
- added copper zone on In2.Cu, net Net-(F4-Pad2)
- added copper zone on F.Cu, net Net-(F5-Pad2)
- added copper zone on In1.Cu, net Net-(F5-Pad2)
- added copper zone on In2.Cu, net Net-(F5-Pad2)
- added copper zone on F.Cu, net Net-(F6-Pad2)
- added copper zone on In1.Cu, net Net-(F6-Pad2)
- added copper zone on In2.Cu, net Net-(F6-Pad2)
- added copper zone on F.Cu, net Net-(F7-Pad2)
- added copper zone on In1.Cu, net Net-(F7-Pad2)
- added copper zone on In2.Cu, net Net-(F7-Pad2)
- added copper zone on F.Cu, net Net-(F8-Pad2)
- added copper zone on In1.Cu, net Net-(F8-Pad2)
- added copper zone on In2.Cu, net Net-(F8-Pad2)
Other:
- board size 240 x 50 mm -> 101 x 50 mm
- board text added: "+"
- board text added: "-"
- board text added: "0.5A PPTC"
- board text added: "BQ"
- board text added: "CELL0"
- board text added: "CELL1"
- board text added: "CELL10"
- board text added: "CELL11"
- board text added: "CELL12"
- board text added: "CELL13"
- board text added: "CELL2"
- board text added: "CELL3"
- board text added: "CELL4"
- board text added: "CELL5"
- board text added: "CELL6"
- board text added: "CELL7"
- board text added: "CELL8"
- board text added: "CELL9"
- board text added: "COML"
- board text added: "COMP"
- board text added: "CURR SENSE MAX 1.5V"
- board text added: "Cell ballance"
- board text added: "FILTER"
- board text added: "GND"
- board text added: "POWER"
- board text added: "STATUS"
- board text added: "THERMISTORS"
- board text added: "VCC"

Commit message: Prace nad masterem
Parts:
- added H1: MountingHole, MountingHole:MountingHole_3.2mm_M3_DIN965, F.Cu at (73.5, 114.0)
- added H2: MountingHole, MountingHole:MountingHole_3.2mm_M3_DIN965, F.Cu at (158.0, 71.5)
- J5: footprint Connector_JST:JST_PHD_B16B-PHDSS_2x08_P2.00mm_Vertical -> Connector_JST:JST_PHD_S16B-PHDSS_2x08_P2.00mm_Horizontal
- moved F19 21.6 mm to (141.0, 81.0), turned to -90 degrees
- moved F24 21.2 mm to (155.5, 104.2), turned to 0 degrees
- moved F20 17.9 mm to (141.5, 77.5), turned to -90 degrees
- moved F23 15.6 mm to (155.5, 102.2), turned to 0 degrees
- moved F22 12.6 mm to (159.0, 104.2), turned to 180 degrees
- moved F21 6.91 mm to (159.0, 102.2), turned to 180 degrees
- moved J13 4.25 mm to (157.0, 80.0), turned to 180 degrees
- moved R3 3.00 mm to (140.5, 84.5)
- moved R6 3.00 mm to (142.0, 84.5)
- moved J5 1.47 mm to (156.8, 98.5)
Routing:
- net GND: track 251.0 -> 212.6 mm, vias 176 -> 168
- net Net-(F19-Pad2): track 31.6 -> 1.74 mm, vias 2 -> 0
- net Net-(J13-Pin_2): track 6.14 -> 33.4 mm, vias 0 -> 1
- net Net-(J5-Pin_15): track 5.28 -> 29.7 mm, vias 0 -> 1
- net Net-(J13-Pin_1): track 3.25 -> 26.8 mm, vias 0 -> 1
- net Net-(F20-Pad2): track 27.2 -> 5.44 mm, vias 2 -> 0
- net Net-(J5-Pin_13): track 5.28 -> 21.3 mm, vias 0 -> 1
- net Net-(J5-Pin_11): track 5.28 -> 12.7 mm
- net Net-(U1-BBN): track 10.1 -> 7.10 mm
- net Net-(U1-BBP): track 8.74 -> 5.74 mm
- net /Temperature/Thermistor6/Thermistor: track 11.2 -> 14.0 mm
- net /Temperature/Thermistor7/Thermistor: track 10.5 -> 13.2 mm
- net /Temperature/Thermistor5/Thermistor: track 12.4 -> 14.6 mm
- net /Temperature/Thermistor3/Thermistor: track 14.3 -> 16.2 mm
- net /Temperature/Thermistor2/Thermistor: track 15.4 -> 17.3 mm
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Other:
- board size 101 x 50 mm -> 92.5 x 57 mm
- board text added: "B2B-PH-K-S-GW"
- board text added: "BMS 2.0 SLAVE BY WIKTOR KRAKOWSKI 2026"
- board text added: "BMS SLAVE 2.0 2026 BY WIKTOR KRAKOWSKI"
