File: BMS_Slave/BMS_Slave.kicad_sch (KiCad schematic)
At the start: 29 parts, among them J33 Dsub 9, J34 Dsub 9, Q8 FZT653TA, T2 TM0608SR, T3 TM0608SR, U1 BQ79614PAPRQ1

Commit message: Dodano connectory hińskie zamiast padów, kontynuacja layoutu
Parts:
- removed J33, J34: Dsub 9, Connector_Dsub:DSUB-9_Pins_Vertical_P2.77x2.84mm_MountingHoles, symbol Connector_Generic:Conn_01x09
- added F19, F20: 0.5A resetable, Fuse:Fuse_0805_2012Metric, symbol Device:Fuse_Small
- added J13, J3, J4: B2B-PH-K-S-GW, Model:CONN2_B2B-PH-K-S_JST, symbol Connector_Generic:Conn_01x02
- added R3, R6: 300, Resistor_SMD:R_0603_1608Metric, symbol Device:R_Small
Connections:
- net GND_HV is gone; now on net GND: U1.36 (REFHM), U1.46 (CVSS), U1.50 (DVSS)
- net dp1+: now reaches T2.3 (PRI_3)
- net dp1+: now also J3.1 (Pin_1)
- net dp1-: now reaches T2.1 (PRI_1)
- net dp1-: now also J3.2 (Pin_2)
- net at U1.63 (BBN): now also R6.1
- net at U1.64 (BBP): now also R3.1
- net dp6-: now reaches T3.3 (PRI_3)
- net dp6-: now also J4.2 (Pin_2)
- net dp6+: now reaches T3.1 (PRI_1)
- net dp6+: now also J4.1 (Pin_1)
- net IIC+ renamed dp3+
- net dp3+: no longer C49.1, R58.2, R75.1, U1.40 (COMLP)
- net IIC- renamed dp3-
- net dp3-: no longer C48.1, R58.1, R76.2, U1.41 (COMLN)
- net ILC+ renamed dp5+
- net dp5+: no longer R78.2, T2.6 (SEC_3)
- net ILC- renamed dp5-
- net dp5-: no longer R79.1, T2.4 (SEC_1)
- new net: F20.2, R6.2
- new net: F20.1, J13.1 (Pin_1)
- new net: F19.1, J13.2 (Pin_2)
- new net: F19.2, R3.2
- new net dp2+: R78.2, T2.4 (SEC_1)
- new net dp2-: R79.1, T2.6 (SEC_3)
- new net dp4+: C49.1, R58.2, R75.1, U1.40 (COMLP)
- new net dp4-: C48.1, R58.1, R76.2, U1.41 (COMLN)
- no-connect marks 24 -> 8
Other:
- sheet Temperature_LTC_1 renamed Temperature
- sheet Temperature: file Temperature_LTC_1.kicad_sch -> Temperature.kicad_sch
- moved on the sheet: C51, C52, C53, R77, R78, R79, T2

Commit message: Zostały małe poprawki na silkscreenie i otwory montażowe
Connections:
- net Battery/Batt1_+ renamed Battery/Batt+
Other:
- sheet Battery ports: added Batt+; removed Batt1_+
Changed lines of the file:
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@@
-			)
-		)
-		(pin "Batt1_+" input
-			(at 59.69 104.14 0)
-			(effects
-				(font
-					(size 1.27 1.27)
-				)
-				(justify right)
 			)
 		)
@@
 			)
 		)
+		(pin "Batt+" output
+			(at 59.69 104.14 0)
+			(effects
+				(font
+					(size 1.27 1.27)
+				)
+				(justify right)
+			)
+		)

Commit message: Prace nad masterem
Parts:
- added H1, H2: MountingHole, MountingHole:MountingHole_3.2mm_M3_DIN965, symbol Mechanical:MountingHole
Changed lines of the file:
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@@
+	)
+	(symbol
+		(lib_id "Mechanical:MountingHole")
+		(at 262.89 24.13 0)
+		(unit 1)
+		(body_style 1)
+		(exclude_from_sim no)
+		(in_bom no)
+		(on_board yes)
+		(in_pos_files yes)
+		(dnp no)
+		(fields_autoplaced yes)
+		(property "Reference" "H1"
+			(at 266.065 22.8599 0)
+			(show_name no)
+			(do_not_autoplace no)
+			(effects
+				(font
+					(size 1.27 1.27)
+				)
+				(justify left)
+			)
+		)
+		(property "Value" "MountingHole"
+			(at 266.065 25.3999 0)
+			(show_name no)
+			(do_not_autoplace no)
+			(effects
+				(font
+					(size 1.27 1.27)
+				)
+				(justify left)
+			)
+		)
+		(property "Footprint" "MountingHole:MountingHole_3.2mm_M3_DIN965"
+			(at 262.89 24.13 0)
+			(hide yes)
+			(show_name no)
+			(do_not_autoplace no)
+			(effects
+				(font
+					(size 1.27 1.27)
+				)
+			)
+		)
+		(property "Datasheet" ""
+			(at 262.89 24.13 0)
+			(hide yes)
+			(show_name no)
+			(do_not_autoplace no)
+			(effects
+				(font
+					(size 1.27 1.27)
+				)
+			)
+		)
+		(property "Description" "Mounting Hole without connection"
+			(at 262.89 24.13 0)
+			(hide yes)
+			(show_name no)
+			(do_not_autoplace no)
+			(effects
+				(font
+					(size 1.27 1.27)
+				)
+			)
+		)
+		(instances
+			(project "BMS_Slave"
+				(path "/5ef38d78-c36e-4401-b313-d3049d9eb692"
+					(reference "H1")
+					(unit 1)
+				)
+			)
+		)
+	)
+	(symbol
+		(lib_id "Mechanical:MountingHole")
+		(at 262.89 31.75 0)
+		(unit 1)
+		(body_style 1)
+		(exclude_from_sim no)
+		(in_bom no)
+		(on_board yes)
+		(in_pos_files yes)
+		(dnp no)
+		(fields_autoplaced yes)
+		(property "Reference" "H2"
+			(at 266.065 30.4799 0)
+			(show_name no)
+			(do_not_autoplace no)
+			(effects
+				(font
+					(size 1.27 1.27)
+				)
+				(justify left)
+			)
+		)
+		(property "Value" "MountingHole"
+			(at 266.065 33.0199 0)
+			(show_name no)
+			(do_not_autoplace no)
+			(effects
+				(font
+					(size 1.27 1.27)
+				)
+				(justify left)
+			)
+		)
+		(property "Footprint" "MountingHole:MountingHole_3.2mm_M3_DIN965"
+			(at 262.89 31.75 0)
+			(hide yes)
+			(show_name no)
+			(do_not_autoplace no)
+			(effects
+				(font
+					(size 1.27 1.27)
+				)
+			)
+		)
+		(property "Datasheet" ""
+			(at 262.89 31.75 0)
+			(hide yes)
+			(show_name no)
+			(do_not_autoplace no)
+			(effects
+				(font
+					(size 1.27 1.27)
+				)
+			)
+		)
+		(property "Description" "Mounting Hole without connection"
+			(at 262.89 31.75 0)
+			(hide yes)
+			(show_name no)
+			(do_not_autoplace no)
+			(effects
+				(font
+					(size 1.27 1.27)
+				)
+			)
+		)
+		(instances
+			(project "BMS_Slave"
+				(path "/5ef38d78-c36e-4401-b313-d3049d9eb692"
+					(reference "H2")
+					(unit 1)
+				)
+			)
+		)
 	)
 	(symbol
