File: BMS_Slave/Temperature.kicad_sch (KiCad schematic)
At the start: 0 parts

Commit message: Zostały małe poprawki na silkscreenie i otwory montażowe
Parts:
- added D1: Red, LED_SMD:LED_0603_1608Metric, symbol Device:LED_Small
- added F21, F22, F23, F24: 0.5A resetable, Fuse:Fuse_0805_2012Metric, symbol Device:Fuse_Small
- added J5: C66560, Connector_JST:JST_PHD_B16B-PHDSS_2x08_P2.00mm_Vertical, symbol Connector_Generic:Conn_02x08_Counter_Clockwise
- added R1: 1k, Resistor_SMD:R_0603_1608Metric, symbol Device:R_Small
Connections:
- net T1: now also D1.1 (K)
- net TSREF: now also R1.2
- new net: F22.1, J5.11 (Pin_11), J5.12 (Pin_12)
- new net: F21.1, J5.10 (Pin_10), J5.9 (Pin_9)
- new net: F23.1, J5.13 (Pin_13), J5.14 (Pin_14)
- new net: F24.1, J5.15 (Pin_15), J5.16 (Pin_16)
- new net: D1.2 (A), R1.1
- new net GND: F21.2, F22.2, F23.2, F24.2
- new net Thermistor/Thermistor: J5.8 (Pin_8)
- new net Thermistor1/Thermistor: J5.7 (Pin_7)
- new net Thermistor2/Thermistor: J5.6 (Pin_6)
- new net Thermistor3/Thermistor: J5.5 (Pin_5)
- new net Thermistor4/Thermistor: J5.4 (Pin_4)
- new net Thermistor5/Thermistor: J5.3 (Pin_3)
- new net Thermistor6/Thermistor: J5.2 (Pin_2)
- new net Thermistor7/Thermistor: J5.1 (Pin_1)
Other:
- sheet Thermistor ports: added Thermistor; removed none
- sheet Thermistor1 ports: added Thermistor; removed none
- sheet Thermistor2 ports: added Thermistor; removed none
- sheet Thermistor3 ports: added Thermistor; removed none
- sheet Thermistor4 ports: added Thermistor; removed none
- sheet Thermistor5 ports: added Thermistor; removed none
- sheet Thermistor6 ports: added Thermistor; removed none
- sheet Thermistor7 ports: added Thermistor; removed none

Commit message: Prace nad masterem
Parts:
- J5: footprint Connector_JST:JST_PHD_B16B-PHDSS_2x08_P2.00mm_Vertical -> Connector_JST:JST_PHD_S16B-PHDSS_2x08_P2.00mm_Horizontal
Changed lines of the file:
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@@
 			)
 		)
-		(property "Footprint" "Connector_JST:JST_PHD_B16B-PHDSS_2x08_P2.00mm_Vertical"
+		(property "Footprint" "Connector_JST:JST_PHD_S16B-PHDSS_2x08_P2.00mm_Horizontal"
 			(at 149.86 98.425 0)
 			(hide yes)
